File: kicad/SnarkBarker.kicad_pcb (KiCad board)
At the start: 2 copper layers, 231.1 x 106.7 mm, 199 parts, among them J1 Bus_ISA_8bit, J2 Bracket Mount, P1 Joystick/MIDI, P2 L7809, T1 2N3904, T2 2N3904, U1 NE558, U10 YM3014B, U11 NJM3403A, U12 MC1408_DIP, U13 805X, U14 SAA1099, U15 SAA1099, U16 74LS08, U17 74LS139, U18 74LS374, U19 74LS374, U2 74LS245, U20 74LS74, U21 74LS125, U22 74LS74, U23 74LS74, U24 74LS32, U25 74LS08, U26 74LS74, U27 74LS32, U28 74LS08, U29 74LS14, U3 74LS244, U30 74LS32, U4 TEA2025B, U5 LM324, U6 LM393, U7 74LS138, U8 74LS138, U9 YM3812

Commit message: finalized the migration to kicad 9
Parts:
- removed C1, C14, C42, C43, C46: 10uF 16V, SoundBlaster:SB_C_RADIAL_75_150
- removed C10, C47, C48, C5, C56, C6, C8, C83, C9: 0.1u, SoundBlaster:SB_C_AXIAL_275
- removed C11, C4: 470uF 16V, SoundBlaster:SB_C_RADIAL_100_320
- removed C12, C15, C17, C18, C3, C7: 100uF 16V, SoundBlaster:SB_C_RADIAL_100_320
- removed C13, C2: 47uF 16V, SoundBlaster:SB_C_RADIAL_75_150
- removed C20, C21, C22, C24, C25, C26, C27, C28, C29: 0.01u, SoundBlaster:SB_C_DISC_200
- removed C36, C37, C49, C54: 1000p, SoundBlaster:SB_C_DISC_200
- removed DRQ1: DMA ENABLE JUMPER, SoundBlaster:SB_HDR_1X2
- removed G*** (x2): LOGO, SoundBlaster:Snark_Barker
- removed IRQ2, IRQ3, IRQ5, IRQ7: Conn_02x01, SoundBlaster:SB_HDR_1X2
- removed L1, L2, L3: ?, SoundBlaster:SB_L_AXIAL_500
- removed MIC1: Microphone, SoundBlaster:SB_MJ-3536N
- removed P1: Joystick/MIDI, SoundBlaster:SB_DB15_152-3415
- removed P2: L7809, SoundBlaster:SB_TO220
- removed REF** (x2): SB_NPTH_110, SoundBlaster:SB_NPTH_110
- removed REF**: MNT_KEYSTONE_9200, Conn:MNT_KEYSTONE_9200
- removed REF***: WEEE-Logo_8.4x12mm_SilkScreen, Symbols:WEEE-Logo_8.4x12mm_SilkScreen
- removed RP1: 2.2K, SoundBlaster:SB_RP_4B
- removed RP2, RP3: 1K, SoundBlaster:SB_RP_4C
- removed RXD1, TXD1: Conn_01x03, SoundBlaster:SB_HDR_1X3
- removed S1: OUT, SoundBlaster:SB_SJ1-3553
- removed S2: ALPS_RK08H_DUAL, SoundBlaster:SB_ALPS_RK08_DUAL
- removed XTL1: 12MHz, SoundBlaster:SB_XTAL_HC49U_RA
- removed ZD1, ZD2, ZD3: 5.1V, SoundBlaster:SB_D_AXIAL_400_ALT
- added C100: 10uF, Capacitor_SMD:C_1210_3225Metric, F.Cu at (235.6, -17.4)
- added C101: 10uF, Capacitor_SMD:C_1210_3225Metric, F.Cu at (235.6, -13.2)
- added C102: 1µF, Capacitor_SMD:C_0805_2012Metric, F.Cu at (290.4, -59.3)
- added C103: 1µF, Capacitor_SMD:C_0805_2012Metric, F.Cu at (290.4, -56.3)
- added C104: 1µF, Capacitor_SMD:C_0805_2012Metric, F.Cu at (294.9, -71.4)
- added C105: 100µF 25V, Capacitor_SMD:CP_Elec_6.3x5.2, F.Cu at (284.9, -25.5)
- added C106: 100µF 25V, Capacitor_SMD:CP_Elec_6.3x5.2, F.Cu at (284.9, -17.4)
- added C107: 100pF, Capacitor_SMD:C_0805_2012Metric, F.Cu at (294.9, -68.4)
- added C108: 100pF, Capacitor_SMD:C_0805_2012Metric, F.Cu at (294.9, -65.3)
- added C90: 150nF, Capacitor_SMD:C_0805_2012Metric, F.Cu at (286.0, -71.4)
- added C91: 22nF, Capacitor_SMD:C_0805_2012Metric, F.Cu at (286.0, -68.4)
- added C92: 22nF, Capacitor_SMD:C_0805_2012Metric, F.Cu at (286.0, -65.3)
- added C93: 150nF, Capacitor_SMD:C_0805_2012Metric, F.Cu at (286.0, -62.3)
- added C94: 150nF, Capacitor_SMD:C_0805_2012Metric, F.Cu at (286.0, -59.3)
- added C95: 150nF, Capacitor_SMD:C_0805_2012Metric, F.Cu at (286.0, -56.3)
- added C96: 22nF, Capacitor_SMD:C_0805_2012Metric, F.Cu at (290.4, -71.4)
- added C97: 150nF, Capacitor_SMD:C_0805_2012Metric, F.Cu at (290.4, -68.4)
- added C98: 100nF, Capacitor_SMD:C_0805_2012Metric, F.Cu at (290.4, -65.3)
- added C99: 100nF, Capacitor_SMD:C_0805_2012Metric, F.Cu at (290.4, -62.3)
- added J4: SPKOUT, Connector_Audio:Jack_3.5mm_CUI_SJ1-3535NG_Horizontal, F.Cu at (200.6, 75.8)
- added J5: IRQ, Connector_PinHeader_2.54mm:PinHeader_2x04_P2.54mm_Vertical, F.Cu at (131.5, 123.7)
- added J6: SPKOUT, Connector_Audio:Jack_3.5mm_CUI_SJ1-3535NG_Horizontal, F.Cu at (200.6, 85.2)
- added JP2: DMA EN, Connector_PinHeader_2.54mm:PinHeader_1x02_P2.54mm_Vertical, F.Cu at (292.5, -14.1)
- added R45: 47, Resistor_SMD:R_0805_2012Metric, F.Cu at (268.5, -16.3)
- added R46: 2k, Resistor_SMD:R_0805_2012Metric, F.Cu at (268.5, -13.4)
- added R47: 2k, Resistor_SMD:R_0805_2012Metric, F.Cu at (268.5, -10.4)
- added R48: 2k, Resistor_SMD:R_0805_2012Metric, F.Cu at (273.0, -28.1)
- added R49: 2k, Resistor_SMD:R_0805_2012Metric, F.Cu at (273.0, -25.2)
- added R50: 20K, Resistor_SMD:R_0805_2012Metric, F.Cu at (273.0, -22.2)
- added R51: 1K, Resistor_SMD:R_0805_2012Metric, F.Cu at (273.0, -19.3)
- added R52: 20K, Resistor_SMD:R_0805_2012Metric, F.Cu at (273.0, -16.3)
- added R53: 1K, Resistor_SMD:R_0805_2012Metric, F.Cu at (273.0, -13.4)
- added R55: 1K, Resistor_SMD:R_0805_2012Metric, F.Cu at (273.0, -10.4)
- added R56: 1K, Resistor_SMD:R_0805_2012Metric, F.Cu at (277.4, -28.1)
- added R57: 0, Resistor_SMD:R_0805_2012Metric, F.Cu at (277.4, -25.2)
- added R58: 0, Resistor_SMD:R_0805_2012Metric, F.Cu at (277.4, -22.2)
- added U31: L7805, Package_TO_SOT_THT:TO-220-3_Horizontal_TabDown, F.Cu at (181.9, 49.1)
- added U32: L7905, Package_TO_SOT_THT:TO-220-3_Horizontal_TabDown, F.Cu at (193.5, 49.1)
- added Y1: 12MHz, Crystal:Crystal_HC49-U_Vertical, F.Cu at (289.1, -33.8)
- C16, C19, C33, C34, C50, C53, C69, C70, C71, C72, C73, C74, C75, C76, C77, C80, C81, C82, C84, C85, C86, C89: footprint SoundBlaster:SB_C_AXIAL_275 -> Capacitor_SMD:C_0805_2012Metric
- C23, C31, C32, C35, C51, C52, C57, C58, C59, C60, C61, C62, C63, C64, C65, C66, C67, C68, C78, C79: footprint SoundBlaster:SB_C_DISC_200 -> Capacitor_SMD:C_0805_2012Metric
- C30, C38, C39, C87, C88: footprint SoundBlaster:SB_C_RADIAL_75_150 -> Capacitor_SMD:C_1210_3225Metric
- C40: footprint SoundBlaster:SB_C_RADIAL_100_320 -> Capacitor_SMD:C_1210_3225Metric
- C41: value 47 -> 47p; footprint SoundBlaster:SB_C_DISC_200 -> Capacitor_SMD:C_0805_2012Metric
- C44, C45, C55: value 10uF 16V -> 10uF; footprint SoundBlaster:SB_C_RADIAL_75_150 -> Capacitor_SMD:C_1210_3225Metric
- D1, D2: footprint SoundBlaster:SB_D_AXIAL_400 -> Diode_SMD:D_0805_2012Metric
- IO1: footprint SoundBlaster:SB_HDR_2X6 -> Connector_PinHeader_2.54mm:PinHeader_2x06_P2.54mm_Vertical
- J1: value Bus_ISA_8bit -> 8-bit ISA slot; footprint SoundBlaster:BUS_PC -> SB:ISA card edge
- J2: value Bracket Mount -> GAME; footprint SoundBlaster:SB_MH_125 -> Connector_Dsub:DSUB-15_Pins_Horizontal_P2.77x2.84mm_EdgePinOffset7.70mm_Housed_MountingHolesOffset9.12mm
- JP1: footprint SoundBlaster:SB_HDR_1X2 -> Connector_PinHeader_2.54mm:PinHeader_1x02_P2.54mm_Vertical
- R1, R2: value 270 -> 10K; footprint SoundBlaster:SB_R_AXIAL_400 -> Resistor_SMD:R_0805_2012Metric
- R10, R11, R12, R13, R14, R15, R16, R17, R22, R25, R26, R27, R28, R29, R30, R31, R32, R33, R35, R36, R37, R39, R41, R42, R43, R44, R5, R6, R7, R8, R9: footprint SoundBlaster:SB_R_AXIAL_400 -> Resistor_SMD:R_0805_2012Metric
- R18: value 1.5K 1% -> 1.5K; footprint SoundBlaster:SB_R_AXIAL_400 -> Resistor_SMD:R_0805_2012Metric
- R19, R20: value 390 -> 20K; footprint SoundBlaster:SB_R_AXIAL_400 -> Resistor_SMD:R_0805_2012Metric
- R21: value 390 -> 1K; footprint SoundBlaster:SB_R_AXIAL_400 -> Resistor_SMD:R_0805_2012Metric
- R23, R3, R34, R4, R40: value 10K -> 1K; footprint SoundBlaster:SB_R_AXIAL_400 -> Resistor_SMD:R_0805_2012Metric
- R24: value 10K -> 4.7K; footprint SoundBlaster:SB_R_AXIAL_400 -> Resistor_SMD:R_0805_2012Metric
- R38: value 2.70K 1% -> 2.7K; footprint SoundBlaster:SB_R_AXIAL_400 -> Resistor_SMD:R_0805_2012Metric
- T1, T2: footprint SoundBlaster:SB_TO92 -> Package_TO_SOT_SMD:SOT-23
- U1: value NE558 -> AT89LP51; footprint SoundBlaster:SB_DIP16_300 -> Package_QFP:TQFP-44_10x10mm_P0.8mm
- U10: value YM3014B -> YM3014; footprint SoundBlaster:SB_DIP8_300 -> Package_DIP:DIP-8_W7.62mm
- U11: value NJM3403A -> LM324; footprint SoundBlaster:SB_DIP14_300 -> Package_SO:SOIC-14_3.9x8.7mm_P1.27mm
- U12: value MC1408_DIP -> MC1408; footprint SoundBlaster:SB_DIP16_300 -> Package_SO:SOIC-16_3.9x9.9mm_P1.27mm
- U13: value 805X -> NE558; footprint SoundBlaster:SB_DIP40_600 -> Package_SO:SOIC-16_4.55x10.3mm_P1.27mm
- U14, U15: footprint SoundBlaster:SB_DIP18_300 -> Package_DIP:DIP-18_W7.62mm
- U16, U20, U21, U22, U23, U24, U25, U26, U27, U28, U29, U30, U5: footprint SoundBlaster:SB_DIP14_300 -> Package_SO:SOIC-14_3.9x8.7mm_P1.27mm
- U17, U7, U8: footprint SoundBlaster:SB_DIP16_300 -> Package_SO:SOIC-16_3.9x9.9mm_P1.27mm
- U18, U19, U2: footprint SoundBlaster:SB_DIP20_300 -> Package_SO:SOIC-20W_7.5x12.8mm_P1.27mm
- U3: value 74LS244 -> 74LS245; footprint SoundBlaster:SB_DIP20_300 -> Package_SO:SOIC-20W_7.5x12.8mm_P1.27mm
- U4: value TEA2025B -> LM4880MX; footprint SoundBlaster:SB_DIP16_300 -> Package_SO:SO-8_3.9x4.9mm_P1.27mm
- U6: footprint SoundBlaster:SB_DIP8_300 -> Package_SO:SOIC-8_3.9x4.9mm_P1.27mm
- U9: footprint SoundBlaster:SB_DIP24_600 -> Package_DIP:DIP-24_W15.24mm
- moved U28 283.8 mm to (316.6, 78.8)
- moved U20 280.3 mm to (334.8, 78.8)
- moved U29 277.0 mm to (306.8, 92.9)
- moved C71 232.7 mm to (204.6, -48.3), turned to 0 degrees
- moved C72 214.0 mm to (204.6, -45.3), turned to 0 degrees
- moved C70 197.1 mm to (200.1, -24.2), turned to 0 degrees
- moved C73 192.0 mm to (204.6, -42.3), turned to 0 degrees
- moved C76 189.4 mm to (204.6, -33.2), turned to 0 degrees
- moved C69 179.1 mm to (200.1, -27.2), turned to 0 degrees
- moved C68 177.8 mm to (200.1, -30.2)
- moved C88 175.6 mm to (208.1, -53.7), turned to 0 degrees
- moved C87 175.6 mm to (208.1, -57.9)
- moved R6 174.6 mm to (109.0, -69.0), turned to 0 degrees
- moved R7 174.4 mm to (109.0, -66.0), turned to 0 degrees
- moved R8 174.2 mm to (109.0, -63.1), turned to 0 degrees
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Connections:
- net /1xx000xxxx renamed Net-(U17A-E)
- net /CLK_14M318 renamed /CLK
- net /CLK_3M579 renamed /CLK/4
- net /CLK_7M159 renamed /CLK/2
- net /CMS1-6_~{CS} renamed /CMS0
- net /CMS7-12_~{CS} renamed /CMS1
- net /DIGITAL_OUT renamed /DSPOUT
- net /IO_READY renamed /IORDY
- net /OPL2 renamed /FMOUT
- net /SAA_L renamed Net-(C60-Pad1)
- net /SAA_R renamed Net-(C58-Pad1)
- net /~{100jjjxxxx} renamed Net-(U17B-O0)
- net /~{111000xxxx} renamed Net-(U17A-O3)
- net /~{CARD_SELECTED} renamed /~{CS}
- net Net-(C55-Pad1) renamed /RB
- net Net-(IO1-Pad1) renamed /IO210
- net Net-(IO1-Pad11) renamed /IO260
- net Net-(IO1-Pad3) renamed /IO220
- net Net-(IO1-Pad5) renamed /IO230
- net Net-(IO1-Pad7) renamed /IO240
- net Net-(IO1-Pad9) renamed /IO250
- net Net-(U10-Pad8) renamed /MP
- C16 pad 1: +12V -> -12V
- C16 pad 2: GNDA -> GND
- C19 pad 1: +9VA -> -5V
- C19 pad 2: GNDA -> GND
- C23 pad 1: Net-(C23-Pad1) -> GND
- C23 pad 2: GNDA -> Net-(U13-CV)
- C32 pad 1: GNDA -> GND
- C33 pad 1: -5VA -> -5V
- C33 pad 2: GNDA -> GND
- C34 pad 2: GNDA -> GND
- C35 pad 2: GNDA -> GND
- C39 pad 2: GNDA -> GND
- C40 pad 1: Net-(C40-Pad1) -> Net-(U6A--)
- C41 pad 1: Net-(C40-Pad1) -> Net-(U6A--)
- C44 pad 1: GNDA -> GND
- C44 pad 2: -5VA -> -5V
- C45 pad 2: GNDA -> GND
- C50 pad 1: -5VA -> -5V
- C50 pad 2: GNDA -> GND
- C52 pad 1: GNDA -> GND
- C53 pad 2: GNDA -> GND
- C55 pad 2: GNDA -> GND
- C57 pad 2: GNDA -> GND
- C58 pad 2: GNDA -> GND
- C59 pad 1: Net-(C59-Pad1) -> Net-(U12-COMPEN)
- C60 pad 2: GNDA -> GND
- C61 pad 1: Net-(C61-Pad1) -> GND
- C61 pad 2: GND -> Net-(U1-XTAL2)
- C62 pad 1: Net-(C62-Pad1) -> GND
- C62 pad 2: GND -> Net-(U1-XTAL1)
- C63 pad 1: Net-(C63-Pad1) -> /OUTR
- C63 pad 2: GNDA -> GND
- C78 pad 1: Net-(C78-Pad1) -> /OUTL
- C78 pad 2: GNDA -> GND
- C81 pad 1: VDDA -> VCC
- C81 pad 2: GNDA -> GND
- C82 pad 1: VDDA -> VCC
- C82 pad 2: GNDA -> GND
- C86 pad 2: GNDA -> GND
- C87 pad 1: VDDA -> VCC
- C87 pad 2: GNDA -> GND
- C89 pad 2: GNDA -> GND
- D1 pad 2: GNDA -> GND
- J1 pad 1: GNDA -> GND
- J1 pad 10: (no net) -> unconnected-(J1-GND-Pad10)
- J1 pad 11: (no net) -> unconnected-(J1-~{SMEMW}-Pad11)
- J1 pad 12: (no net) -> unconnected-(J1-~{SMEMR}-Pad12)
- J1 pad 15: (no net) -> unconnected-(J1-~{DACK3}-Pad15)
- J1 pad 16: (no net) -> unconnected-(J1-DRQ3-Pad16)
- J1 pad 19: (no net) -> unconnected-(J1-~{DACK0}-Pad19)
- J1 pad 2: /BUSRESET -> /RST
- J1 pad 20: (no net) -> unconnected-(J1-CLK-Pad20)
- J1 pad 22: (no net) -> unconnected-(J1-IRQ6-Pad22)
- J1 pad 24: (no net) -> unconnected-(J1-IRQ4-Pad24)
- J1 pad 26: (no net) -> unconnected-(J1-~{DACK2}-Pad26)
- J1 pad 27: (no net) -> unconnected-(J1-TC-Pad27)
- J1 pad 28: (no net) -> unconnected-(J1-ALE-Pad28)
- J1 pad 3: VDDA -> VCC
- J1 pad 32: (no net) -> unconnected-(J1-IO-Pad32)
- J1 pad 43: (no net) -> unconnected-(J1-BA19-Pad43)
- J1 pad 44: (no net) -> unconnected-(J1-BA18-Pad44)
- J1 pad 45: (no net) -> unconnected-(J1-BA17-Pad45)
- J1 pad 46: (no net) -> unconnected-(J1-BA16-Pad46)
- J1 pad 47: (no net) -> unconnected-(J1-BA15-Pad47)
- J1 pad 48: (no net) -> unconnected-(J1-BA14-Pad48)
- J1 pad 49: (no net) -> unconnected-(J1-BA13-Pad49)
- J1 pad 5: (no net) -> unconnected-(J1--5V-Pad5)
- J1 pad 50: (no net) -> unconnected-(J1-BA12-Pad50)
- J1 pad 51: (no net) -> unconnected-(J1-BA11-Pad51)
- J1 pad 52: (no net) -> unconnected-(J1-BA10-Pad52)
- J1 pad 6: (no net) -> unconnected-(J1-DRQ2-Pad6)
- J1 pad 8: (no net) -> unconnected-(J1-UNUSED-Pad8)
- J2 pad 1: GNDA -> /GAME_5V
- JP1 pad 1: Net-(JP1-Pad1) -> Net-(JP1-Pin_1)
- JP1 pad 2: /JOYSTICK_~{CS} -> /~{JOYCS}
- R1 pad 1: Net-(R1-Pad1) -> Net-(U14-IREF)
- R1 pad 2: Net-(C2-Pad1) -> VCC
- R12 pad 2: GNDA -> GND
- R13 pad 2: GNDA -> GND
- R14 pad 1: +5VD -> VCC
- R18 pad 1: Net-(R18-Pad1) -> Net-(U12-I0)
- R19 pad 1: -5VA -> Net-(C102-Pad2)
- R19 pad 2: -12V -> Net-(U4-IN_A)
- R2 pad 1: Net-(R2-Pad1) -> Net-(U15-IREF)
- R2 pad 2: Net-(C13-Pad1) -> VCC
- R20 pad 1: +12V -> Net-(C103-Pad2)
- R20 pad 2: +5VA -> Net-(U4-IN_B)
- R21 pad 1: +12V -> /GAME_DIGITAL3
- R21 pad 2: +5VD -> VCC
- R22 pad 1: Net-(C49-Pad2) -> Net-(C103-Pad1)
- R23 pad 1: Net-(C43-Pad1) -> /GAME_DIGITAL4
- R23 pad 2: Net-(C49-Pad2) -> VCC
- R24 pad 1: Net-(C42-Pad1) -> +5VA
- R24 pad 2: Net-(C54-Pad1) -> Net-(U6A--)
- R25 pad 1: Net-(C54-Pad1) -> Net-(C102-Pad1)
- R28 pad 1: Net-(C54-Pad1) -> Net-(C102-Pad1)
- R29 pad 1: Net-(C54-Pad1) -> Net-(C102-Pad1)
- R3 pad 1: Net-(C37-Pad2) -> /GAME_DIGITAL1
- R3 pad 2: Net-(C43-Pad2) -> VCC
- R30 pad 1: Net-(C49-Pad2) -> Net-(C103-Pad1)
- R31 pad 1: Net-(C49-Pad2) -> Net-(C103-Pad1)
- R32 pad 1: Net-(C63-Pad1) -> /OUTL
- R32 pad 2: +5VD -> VCC
- R33 pad 1: Net-(C78-Pad1) -> /OUTR
- R33 pad 2: +5VD -> VCC
- R34 pad 1: +5VD -> VCC
- R34 pad 2: Net-(R34-Pad2) -> Net-(U13-OUTPUT_D)
- R35 pad 2: Net-(R35-Pad2) -> Net-(U11B--)
- R36 pad 2: Net-(C63-Pad1) -> /OUTR
- R37 pad 2: Net-(C78-Pad1) -> /OUTL
- R38 pad 1: Net-(R38-Pad1) -> Net-(U12-VREF+)
- R38 pad 2: +5VD -> VCC
- R39 pad 1: +5VD -> /DTACK
- R39 pad 2: Net-(R39-Pad2) -> VCC
- R4 pad 1: Net-(C36-Pad1) -> /GAME_DIGITAL2
- R4 pad 2: Net-(C42-Pad2) -> VCC
- R40 pad 1: +5VD -> VCC
- R40 pad 2: Net-(R40-Pad2) -> Net-(U13-OUTPUT_A)
- R42 pad 2: /JOYSTICK_~{CS} -> /~{JOYCS}
- R5 pad 2: GNDA -> GND
- R9 pad 1: Net-(C40-Pad1) -> Net-(U6A--)
- T1 pad 1: GNDA -> GND
- T2 pad 1: GNDA -> GND
- U1 pad 1: Net-(RP2-Pad3) -> /DAC5
- U1 pad 10: Net-(C22-Pad1) -> /~{DMA_EN}
- U1 pad 11: Net-(U1-Pad11) -> /DREQUEST
- U1 pad 12: GNDA -> /~{DSP_WRITE}
- U1 pad 13: /~{IC} -> /~{DSP_READ}
- U1 pad 14: Net-(U1-Pad11) -> Net-(U1-XTAL2)
- U1 pad 15: Net-(C20-Pad1) -> Net-(U1-XTAL1)
- U1 pad 16: Net-(RP2-Pad2) -> GND
- U1 pad 2: Net-(C26-Pad1) -> /DAC6
- U1 pad 3: Net-(U1-Pad11) -> /DAC7
- U1 pad 4: Net-(C23-Pad1) -> /RESET
- U1 pad 5: VDDA -> /MIDI_IN
- U1 pad 6: Net-(U1-Pad11) -> unconnected-(U1-NC-Pad6)
- U1 pad 7: Net-(C21-Pad1) -> /MIDI_OUT
- U1 pad 8: Net-(RP2-Pad4) -> /IREQUEST
- U1 pad 9: Net-(RP2-Pad5) -> /DSP_BUSY
- U10 pad 1: VDDA -> VCC
- U10 pad 2: Net-(U10-Pad2) -> Net-(U10-BUFF)
- U10 pad 6: GNDA -> GND
- U11 pad 10: GNDA -> unconnected-(U11C-+-Pad10)
- U11 pad 11: -5VA -> -5V
- U11 pad 12: Net-(U10-Pad2) -> unconnected-(U11D-+-Pad12)
- U11 pad 13: Net-(R35-Pad2) -> unconnected-(U11D---Pad13)
- U11 pad 14: Net-(R35-Pad2) -> unconnected-(U11-Pad14)
- U11 pad 5: GNDA -> Net-(U10-BUFF)
- U11 pad 6: Net-(C49-Pad2) -> Net-(U11B--)
- U11 pad 7: Net-(C43-Pad1) -> Net-(U11B--)
- U11 pad 8: Net-(C42-Pad1) -> unconnected-(U11-Pad8)
- U11 pad 9: Net-(C54-Pad1) -> unconnected-(U11C---Pad9)
- U12 pad 1: GNDA -> VCC
- U12 pad 10: /DAC2 -> /DAC1
- U12 pad 11: /DAC1 -> /DAC2
- U12 pad 12: /DAC0 -> /DAC3
- U12 pad 13: VDDA -> /DAC4
- U12 pad 14: Net-(R38-Pad1) -> /DAC5
- U12 pad 15: GNDA -> /DAC6
- U12 pad 16: Net-(C59-Pad1) -> /DAC7
- U12 pad 2: GNDA -> Net-(U12-VREF+)
- U12 pad 3: -12V -> GND
- U12 pad 4: Net-(R18-Pad1) -> Net-(U12-COMPEN)
- U12 pad 5: /DAC7 -> unconnected-(U12-NC-Pad5)
- U12 pad 6: /DAC6 -> GND
- U12 pad 7: /DAC5 -> -12V
- U12 pad 8: /DAC4 -> Net-(U12-I0)
- U12 pad 9: /DAC3 -> /DAC0
- U13 pad 1: /DAC0 -> Net-(U13-OUTPUT_A)
- U13 pad 10: Net-(RXD1-Pad3) -> /GAME_ANALOG2
- U13 pad 11: Net-(TXD1-Pad3) -> Net-(U13-TRIGGER_A)
- U13 pad 12: /IREQUEST -> GND
- U13 pad 13: /DSP_BUSY -> /~{IC}
- U13 pad 14: /~{DMA_EN} -> Net-(U13-TRIGGER_A)
- U13 pad 15: /DREQUEST -> /GAME_ANALOG1
- U13 pad 16: /~{DSP_WRITE} -> Net-(U13-OUTPUT_D)
- U13 pad 2: /DAC1 -> /GAME_ANALOG4
- U13 pad 3: /DAC2 -> Net-(U13-TRIGGER_A)
- U13 pad 4: /DAC3 -> Net-(U13-CV)
- U13 pad 5: /DAC4 -> VCC
- U13 pad 6: /DAC5 -> Net-(U13-TRIGGER_A)
- U13 pad 7: /DAC6 -> /GAME_ANALOG3
- U13 pad 8: /DAC7 -> Net-(U13-OUTPUT_B)
- U13 pad 9: /RESET -> Net-(U13-OUTPUT_C)
- U14 pad 18: VDDA -> VCC
- U14 pad 4: Net-(C63-Pad1) -> /OUTR
- U14 pad 5: Net-(C78-Pad1) -> /OUTL
- U14 pad 6: Net-(R34-Pad2) -> Net-(U14-IREF)
- U14 pad 7: Net-(R39-Pad2) -> /DTACK
- U14 pad 9: GNDA -> GND
- U15 pad 18: VDDA -> VCC
- U15 pad 4: Net-(C63-Pad1) -> /OUTR
- U15 pad 5: Net-(C78-Pad1) -> /OUTL
- U15 pad 6: Net-(R40-Pad2) -> Net-(U15-IREF)
- U15 pad 7: Net-(R39-Pad2) -> /DTACK
- U15 pad 9: GNDA -> GND
- U16 pad 11: (no net) -> unconnected-(U16-Pad11)
- U16 pad 12: (no net) -> unconnected-(U16-Pad12)
- U16 pad 13: (no net) -> unconnected-(U16-Pad13)
- U16 pad 4: /~{IOW} -> Net-(R41-Pad2)
- U16 pad 5: Net-(R41-Pad2) -> /~{IOW}
- U17 pad 10: (no net) -> unconnected-(U17B-O2-Pad10)
- U17 pad 11: (no net) -> unconnected-(U17B-O1-Pad11)
- U17 pad 4: /~{100000xxxx} -> Net-(U17A-O0)
- U17 pad 5: (no net) -> unconnected-(U17A-O1-Pad5)
- U17 pad 6: (no net) -> unconnected-(U17A-O2-Pad6)
- U17 pad 9: (no net) -> unconnected-(U17B-O3-Pad9)
- U20 pad 1: Net-(U20-Pad1) -> Net-(U20A-~{R})
- U20 pad 10: Net-(U20-Pad10) -> Net-(U20B-~{S})
- U20 pad 6: (no net) -> unconnected-(U20A-~{Q}-Pad6)
- U20 pad 8: (no net) -> unconnected-(U20B-~{Q}-Pad8)
- U22 pad 6: (no net) -> unconnected-(U22A-~{Q}-Pad6)
- U22 pad 8: (no net) -> unconnected-(U22B-~{Q}-Pad8)
- U24 pad 1: /JOYSTICK_~{CS} -> Net-(U17A-O0)
- U24 pad 10: /~{WR} -> /~{RD}
- U24 pad 12: /DSPRST_~{CS} -> /~{WR}
- U24 pad 13: /~{WR} -> /DSPRST_~{CS}
- U24 pad 2: /~{RD} -> /A3
- U24 pad 3: Net-(U24-Pad3) -> Net-(JP1-Pin_1)
- U24 pad 4: /A3 -> /~{WR}
- U24 pad 5: /~{100000xxxx} -> /~{JOYCS}
- U24 pad 6: Net-(JP1-Pad1) -> Net-(U13-TRIGGER_A)
- U24 pad 8: Net-(U1-Pad11) -> Net-(U3-CE)
- U24 pad 9: /JOYSTICK_~{CS} -> /~{JOYCS}
- U25 pad 10: Net-(R44-Pad2) -> /~{IC}
- U25 pad 2: /JOYSTICK_~{CS} -> /~{JOYCS}
- U25 pad 4: Net-(R39-Pad2) -> Net-(R44-Pad2)
- U25 pad 5: /~{IC} -> /~{IOR}
- U25 pad 6: Net-(U20-Pad10) -> /~{RD}
- U25 pad 8: /~{RD} -> Net-(U20B-~{S})
- U25 pad 9: /~{IOR} -> /DTACK
- U26 pad 13: Net-(U26-Pad13) -> Net-(U26B-~{R})
- U26 pad 5: Net-(U26-Pad5) -> Net-(U26A-Q)
- U26 pad 6: (no net) -> unconnected-(U26A-~{Q}-Pad6)
- U26 pad 8: (no net) -> unconnected-(U26B-~{Q}-Pad8)
- U28 pad 1: /~{RESET} -> /~{RD_DAV}
- U28 pad 10: /~{RESET} -> /DSPRD_~{CS}
- U28 pad 12: /DSPWR_~{CS} -> /~{DMAOUT}
- U28 pad 13: /~{DMAOUT} -> /DSPWR_~{CS}
- U28 pad 2: /~{DMAOUT} -> /~{RESET}
- U28 pad 3: Net-(U20-Pad1) -> Net-(U26B-~{R})
- U28 pad 4: /~{DMAOUT} -> /~{RESET}
- U28 pad 5: /DSPRD_~{CS} -> /~{DMAOUT}
- U28 pad 6: Net-(U27-Pad1) -> Net-(U20A-~{R})
- U28 pad 8: Net-(U26-Pad13) -> Net-(U27-Pad1)
- U28 pad 9: /~{RD_DAV} -> /~{DMAOUT}
- U29 pad 1: /BUSRESET -> /RST
- U29 pad 10: (no net) -> unconnected-(U29-Pad10)
- U29 pad 11: (no net) -> unconnected-(U29-Pad11)
- U29 pad 12: (no net) -> unconnected-(U29-Pad12)
- U29 pad 13: (no net) -> unconnected-(U29-Pad13)
- U29 pad 3: (no net) -> unconnected-(U29-Pad3)
- U29 pad 4: (no net) -> unconnected-(U29-Pad4)
- U3 pad 1: Net-(U24-Pad3) -> GND
- U3 pad 11: /BUTTON1 -> /GAME_DIGITAL4
- U3 pad 12: /D3 -> /GAME_DIGITAL3
- U3 pad 13: /BUTTON2 -> /GAME_DIGITAL2
- U3 pad 14: /D2 -> /GAME_DIGITAL1
- U3 pad 15: /BUTTON4 -> Net-(U13-OUTPUT_A)
- U3 pad 16: /D1 -> Net-(U13-OUTPUT_B)
- U3 pad 17: /BUTTON3 -> Net-(U13-OUTPUT_C)
- U3 pad 18: /D0 -> Net-(U13-OUTPUT_D)
- U3 pad 19: Net-(U24-Pad3) -> Net-(U3-CE)
- U3 pad 2: Net-(RP2-Pad2) -> /D0
- U3 pad 3: /D7 -> /D1
- U3 pad 4: Net-(RP2-Pad5) -> /D2
- U3 pad 5: /D6 -> /D3
- U3 pad 6: Net-(RP2-Pad4) -> /D4
- U3 pad 8: Net-(RP2-Pad3) -> /D6
- U3 pad 9: /D4 -> /D7
- U30 pad 1: /~{DMA_EN} -> Net-(U26A-Q)
- U30 pad 10: /BUSRESET -> /DAV_DSP
- U30 pad 11: (no net) -> unconnected-(U30-Pad11)
- U30 pad 12: (no net) -> unconnected-(U30-Pad12)
- U30 pad 13: (no net) -> unconnected-(U30-Pad13)
- U30 pad 2: /~{DACK1} -> /RST
- U30 pad 3: /~{DMAOUT} -> /RESET
- U30 pad 4: /DSP_BUSY -> /~{DMA_EN}
- U30 pad 5: /DAV_DSP -> /~{DACK1}
- U30 pad 6: Net-(U21-Pad5) -> /~{DMAOUT}
- U30 pad 8: /RESET -> Net-(U21-Pad5)
- U30 pad 9: Net-(U26-Pad5) -> /DSP_BUSY
- U4 pad 1: (no net) -> Net-(U4-OUT_A)
- U4 pad 2: Net-(C12-Pad2) -> Net-(U4-IN_A)
- U4 pad 4: GNDA -> GND
- U4 pad 5: GNDA -> GND
- U4 pad 6: Net-(R2-Pad1) -> Net-(U4-IN_B)
- U4 pad 8: Net-(C15-Pad1) -> +5VA
- U5 pad 10: GNDA -> GND
- U5 pad 11: -5VA -> GND
- U5 pad 14: Net-(C40-Pad1) -> Net-(U6A--)
- U5 pad 9: Net-(R18-Pad1) -> Net-(U12-I0)
- U6 pad 2: Net-(C40-Pad1) -> Net-(U6A--)
- U6 pad 4: GNDA -> GND
- U6 pad 5: GNDA -> GND
- U6 pad 6: GNDA -> GND
- U6 pad 7: (no net) -> unconnected-(U6-Pad7)
- U7 pad 7: (no net) -> unconnected-(U7-O7-Pad7)
- U8 pad 13: (no net) -> unconnected-(U8-O2-Pad13)
- U9 pad 19: (no net) -> unconnected-(U9-NC-Pad19)
- U9 pad 2: (no net) -> unconnected-(U9-~{IRQ}-Pad2)
- U9 pad 22: (no net) -> unconnected-(U9-NC-Pad22)
- U9 pad 8: (no net) -> unconnected-(U9-NC-Pad8)
- U9 pad 9: (no net) -> unconnected-(U9-NC-Pad9)
Routing:
- net GND: track 745.6 -> 0.00 mm, vias 2 -> 0
- net VCC: track 623.0 -> 0.00 mm, vias 3 -> 0
- net GNDA: track 571.2 -> 0.00 mm, vias 7 -> 0
- net /~{IC}: track 321.3 -> 0.00 mm, vias 1 -> 0
- net /BUSRESET: track 306.5 -> 0.00 mm, vias 4 -> 0
- net VDDA: track 292.5 -> 0.00 mm, vias 8 -> 0
- net /~{RD}: track 280.0 -> 0.00 mm, vias 4 -> 0
- net /MIDI_OUT: track 267.9 -> 0.00 mm, vias 1 -> 0
- net /MIDI_IN: track 265.7 -> 0.00 mm, vias 2 -> 0
- net /~{DACK1}: track 245.9 -> 0.00 mm, vias 6 -> 0
- net /D7: track 256.0 -> 24.0 mm, vias 5 -> 0
- net /~{WR}: track 226.9 -> 0.00 mm, vias 4 -> 0
- net /D0: track 284.6 -> 61.4 mm, vias 6 -> 0
- net /IORDY: track 207.7 -> 0.00 mm, vias 3 -> 0
- net +5VD: track 206.9 -> 0.00 mm
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- removed copper zone on F.Cu, net GND
- removed copper zone on B.Cu, net GNDA
- removed copper zone on F.Cu, net GNDA
- removed copper zone on B.Cu, net Net-(C27-Pad1)
- removed copper zone on F.Cu, net Net-(C27-Pad1)
Other:
- board size 231.1 x 106.7 mm -> 103.7 x 109.4 mm
- copper layers 2 -> 4
- rule pad_to_mask_clearance: 0.2 -> 0.038
- board text added: "260h 250h 240h 230h 220h 210h"
- board text added: "IRQ2 IRQ3 IRQ5 IRQ7"
- board text removed: "01/19"
- board text removed: "1"
- board text removed: "210"
- board text removed: "220"
- board text removed: "230"
- board text removed: "240"
- board text removed: "250"
- board text removed: "260"
- board text removed: "31"
- board text removed: "CC BY-SA (Attribution-ShareAlike)"
- board text removed: "CREDITS"
- board text removed: "CT-1320C"
- board text removed: "Foone: testing"
- board text removed: "GND"
- board text removed: "GoodTofuFriday: PCB photography"
- board text removed: "I/O ADDX"
- board text removed: "Lord_Nightmare, balrog, kevtris: lots of info"
- board text removed: "MADE IN ANGER"
- board text removed: "RXD"
- board text removed: "SHOUTS TO cr1901, CommodoreZ, glitch, and Trixter"
- board text removed: "Special thanks to ##yamahasynths"
- board text removed: "TXD"
- board text removed: "TubeTimeUS: PCB reversing and forwarding,"
- board text removed: "VCC"
- board text removed: "also firmware analysis"
- board text removed: "digshadow: misc reversing"
- board text removed: "©"

Commit message: routing
Parts:
- removed U13: NE558, Package_SO:SOIC-16_4.55x10.3mm_P1.27mm
- added C1: 0.01u, Capacitor_SMD:C_0805_2012Metric, F.Cu at (175.5, 97.3)
- added C2: 0.01u, Capacitor_SMD:C_0805_2012Metric, F.Cu at (170.9, 107.6)
- added C3: 0.01u, Capacitor_SMD:C_0805_2012Metric, F.Cu at (170.9, 113.0)
- added U33: NE556, Package_SO:SOIC-14_3.9x8.7mm_P1.27mm, F.Cu at (177.6, 102.4)
- added U34: NE556, Package_SO:SOIC-14_3.9x8.7mm_P1.27mm, F.Cu at (177.6, 110.6)
- C100, C101, C107, C108, C31, C32, C33, C34, C38, C39, C40, C41, C44, C45, C50, C52, C57, C61, C62, C63, C64, C65, C66, C67, C68, C69, C70, C71, C72, C73, C74, C76, C77, C78, C81, C82, C89, C90, C93, C94, C97, D1, D2, R10, R13, R14, R15, R16, R17, R18, R21, R23, R24, R26, R27, R3, R32, R33, R34, R35, R39, R4, R40, R41, R42, R43, R5, R51, R53, R6, R7, R8, R9, T1, T2, U11, U16, U20, U23, U26, U27, U28, U29, U5, U6: moved to B.Cu
- C30: value 10uF 16V -> 10uF
- JP1: value JOYSTICK EN -> Gameport enable
- JP2: value DMA EN -> DMA Enable
- U12: value MC1408 -> DAC0808
- moved C98 217.3 mm to (187.7, 126.1), turned to 90 degrees
- moved JP2 216.4 mm to (100.6, 86.0)
- moved C99 210.7 mm to (187.1, 121.3)
- moved C104 210.1 mm to (160.9, 90.5), turned to 90 degrees
- moved C96 209.8 mm to (187.2, 111.3), turned to 180 degrees
- moved C92 208.8 mm to (186.3, 118.1), turned to 90 degrees
- moved C97 206.2 mm to (197.3, 115.6), turned to 180 degrees
- moved C91 203.2 mm to (187.2, 109.2), turned to 180 degrees
- moved C93 200.5 mm to (197.4, 117.6), turned to 180 degrees
- moved U28 199.4 mm to (118.3, 99.3), turned to -90 degrees
- moved U20 198.9 mm to (139.8, 118.1), turned to -90 degrees
- moved C90 197.0 mm to (197.2, 104.5), turned to 180 degrees
- moved C103 194.3 mm to (166.5, 93.2)
- moved Y1 192.0 mm to (127.7, 70.3), turned to 90 degrees
- moved C102 191.8 mm to (163.1, 84.2), turned to 180 degrees
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Connections:
- J6 pad T: unconnected-(J6-PadT) -> Net-(C30-Pad2)
- R34 pad 2: Net-(U13-OUTPUT_D) -> /TMOUT4
- R40 pad 2: Net-(U13-OUTPUT_A) -> /TMOUT3
- R51 pad 2: Net-(U13-OUTPUT_B) -> /TMOUT2
- R53 pad 2: Net-(U13-OUTPUT_C) -> /TMOUT1
- U24 pad 6: Net-(U13-TRIGGER_A) -> /JOYTMR
- U3 pad 15: Net-(U13-OUTPUT_A) -> /TMOUT4
- U3 pad 16: Net-(U13-OUTPUT_B) -> /TMOUT3
- U3 pad 17: Net-(U13-OUTPUT_C) -> /TMOUT2
- U3 pad 18: Net-(U13-OUTPUT_D) -> /TMOUT1
Routing:
- net -12V: track 0.00 -> 156.2 mm, vias 0 -> 2
- net GND: track 0.00 -> 141.9 mm, vias 0 -> 30
- net +12V: track 0.00 -> 126.3 mm, vias 0 -> 2
- net VCC: track 0.00 -> 120.8 mm, vias 0 -> 26
- net /~{IC}: track 0.00 -> 117.3 mm, vias 0 -> 3
- net /D7: track 24.0 -> 139.0 mm, vias 0 -> 4
- net /MIDI_OUT: track 0.00 -> 111.6 mm
- net /MIDI_IN: track 0.00 -> 103.7 mm
- net /~{WR}: track 0.00 -> 88.2 mm, vias 0 -> 1
- net Net-(U3-CE): track 0.00 -> 84.5 mm, vias 0 -> 2
- net /A0: track 0.00 -> 81.6 mm, vias 0 -> 1
- net /D1: track 28.5 -> 110.1 mm, vias 0 -> 1
- net /~{RD}: track 0.00 -> 81.1 mm
- net /CMS1: track 0.00 -> 75.8 mm, vias 0 -> 1
- net /D2: track 30.3 -> 100.0 mm, vias 0 -> 1
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- added copper zone on In2.Cu, net +5VA
- added copper zone on B.Cu, net GND
- added copper zone on F.Cu, net GND
- added copper zone on In1.Cu, net GND
- added copper zone on In2.Cu, net VCC
Other:
- board size 103.7 x 109.4 mm -> 103.7 x 78 mm

Commit message: routing almost finished
Parts:
- added G1: LOGO, SB:trw_logo, F.Cu at (135.4, 83.2)
- added REF**: pinch, SB:pinch, F.Cu at (181.9, 70.1)
- C33, C34: moved to F.Cu
- J4: footprint Connector_Audio:Jack_3.5mm_CUI_SJ1-3535NG_Horizontal -> SB:TRS jack
- J6: value SPKOUT -> MIC; footprint Connector_Audio:Jack_3.5mm_CUI_SJ1-3535NG_Horizontal -> SB:TRS jack
- moved C66 45.6 mm to (133.2, 72.4), turned to 180 degrees
- moved U20 22.8 mm to (129.7, 97.7)
- moved C33 21.2 mm to (170.9, 79.5), turned to 180 degrees
- moved C34 16.8 mm to (167.2, 79.5)
- moved J4 5.10 mm to (195.6, 85.5)
- moved J6 5.08 mm to (195.7, 76.0)
- moved C3 1.55 mm to (171.8, 111.7), turned to -90 degrees
- moved C30 1.51 mm to (184.2, 78.9)
- moved R41 0.47 mm to (116.2, 109.3)
- moved R7 0.16 mm to (173.9, 74.9)
- moved J2 0.14 mm to (191.5, 119.6)
- moved U12 0.13 mm to (151.5, 67.4)
Connections:
- R14 pad 1: VCC -> +5VA
- U5 pad 11: GND -> -5V
Routing:
- net /~{DACK1}: track 17.2 -> 133.9 mm, vias 0 -> 1
- net /RST: track 1.56 -> 116.9 mm
- net /IORDY: track 10.9 -> 114.4 mm, vias 1 -> 2
- net /~{ISA_WR}: track 3.03 -> 91.5 mm, vias 0 -> 3
- net /~{RESET}: track 16.8 -> 86.7 mm, vias 1 -> 3
- net Net-(U20B-C): track 0.00 -> 66.6 mm, vias 0 -> 2
- net /DRQ1: track 14.5 -> 77.4 mm
- net Net-(U20A-Q): track 0.00 -> 62.8 mm, vias 0 -> 2
- net Net-(U20B-Q): track 0.00 -> 61.5 mm, vias 0 -> 2
- net Net-(J5-Pin_1): track 7.62 -> 64.1 mm, vias 0 -> 1
- net /~{WR}: track 88.2 -> 138.3 mm, vias 1 -> 2
- net Net-(U26A-C): track 0.00 -> 39.5 mm, vias 0 -> 2
- net Net-(U12-I0): track 2.30 -> 36.9 mm, vias 0 -> 1
- net -5V: track 8.06 -> 39.2 mm, vias 0 -> 2
- net /~{IC}: track 117.3 -> 144.1 mm, vias 3 -> 5
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Other:
- board text added: "Mini"
- board text added: "Snark Barker"

Commit message: finalized routing
Parts:
- added J3: Prog, Connector_PinHeader_2.54mm:PinHeader_1x07_P2.54mm_Vertical, F.Cu at (132.1, 61.1)
- added J7: DSP PWR, Connector_PinHeader_2.54mm:PinHeader_1x02_P2.54mm_Vertical, F.Cu at (123.7, 60.8)
- C79: moved to B.Cu
- moved C79 24.0 mm to (107.6, 62.9)
- moved R38 7.17 mm to (152.3, 61.8), turned to 90 degrees
- moved C68 5.50 mm to (136.4, 67.2), turned to 180 degrees
- moved R30 4.03 mm to (170.1, 95.3)
- moved R37 3.83 mm to (170.3, 98.4), turned to -90 degrees
- moved C60 2.80 mm to (173.8, 95.3)
- moved C82 1.98 mm to (117.8, 61.9)
- moved C1 1.64 mm to (173.8, 97.5)
- moved C53 1.31 mm to (150.1, 61.8), turned to 90 degrees
- moved R36 1.27 mm to (158.4, 87.0), turned to -90 degrees
- moved C101 1.18 mm to (186.3, 62.4)
- moved C45 1.17 mm to (186.3, 67.0)
- moved R31 0.93 mm to (166.4, 95.3)
- moved C100 0.70 mm to (163.8, 63.8)
- moved C59 0.53 mm to (155.2, 62.4)
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Connections:
- U1 pad 29: VCC -> VPP
- U1 pad 38: VCC -> VPP
Routing:
- net /JOYTMR: track 14.8 -> 129.7 mm, vias 0 -> 2
- net /~{DMAOUT}: track 11.5 -> 71.6 mm, vias 0 -> 3
- net /~{ISA_RD}: track 16.2 -> 71.3 mm, vias 2 -> 4
- net VPP: track 0.00 -> 33.2 mm, vias 0 -> 2
- net /~{DSP_WRITE}: track 33.2 -> 63.8 mm, vias 0 -> 2
- net /~{DSP_READ}: track 18.8 -> 32.6 mm, vias 0 -> 2
- net /DAC7: track 20.4 -> 31.6 mm
- net /MIDI_IN: track 103.8 -> 114.3 mm
- net Net-(U3-CE): track 84.7 -> 94.3 mm
- net /MIDI_OUT: track 111.6 -> 120.3 mm
- net /DAC4: track 11.2 -> 19.7 mm, vias 0 -> 1
- net /RESET: track 27.6 -> 35.9 mm
- net Net-(U12-VREF+): track 12.7 -> 6.86 mm
- net /DAC6: track 18.1 -> 23.3 mm, vias 0 -> 1
- net GND: track 150.9 -> 145.9 mm, vias 40 -> 46
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Other:
- board size 103.7 x 78 mm -> 103.7 x 78.5 mm

Commit message: finalized first revision
Parts:
- removed R57, R58: 0, Resistor_SMD:R_0805_2012Metric
- added C75: 10uF, Capacitor_SMD:C_1210_3225Metric, F.Cu at (100.8, 95.8)
- C10: renamed from C23; value 0.01u -> 10n
- C11: renamed from C1; value 0.01u -> 10n
- C12: renamed from C2; value 0.01u -> 10n
- C13: renamed from C94; value 150nF -> 100n
- C14: renamed from C90; value 150nF -> 100n
- C15: renamed from C95; value 150nF -> 100n
- C16: renamed from C91; value 22nF -> 22n
- C17: renamed from C96; value 22nF -> 22n
- C18: renamed from C92; value 22nF -> 22n
- C19: renamed from C97; value 150nF -> 100n
- C20: renamed from C93; value 150nF -> 100n
- C21: renamed from C98; value 100nF -> 100n
- C22: renamed from C99; value 100nF -> 100n
- C23: renamed from C57; value 4700p -> 4.7n
- C25: renamed from C63; value 1000p -> 1n
- C26: renamed from C78; value 1000p -> 1n
- C27: renamed from C58; value 2200p -> 2.2n
- C28: renamed from C60; value 2200p -> 2.2n
- C29: renamed from C102; value 1µF -> 1uF
- C30: renamed from C103; value 1µF -> 1uF
- C31: renamed from C104; value 1µF -> 1uF
- C32: renamed from C105; value 100µF 25V -> 100uF
- C33: renamed from C106; value 100µF 25V -> 100uF
- C34: renamed from C107; value 100pF -> 100p
- C35: renamed from C108; value 100pF -> 100p
- C38: renamed from C31; value 1000p -> 1n
- C39: renamed from C38; value 10uF 16V -> 10uF
- C41: renamed from C89; value 0.1u -> 100n
- C42: renamed from C39; value 10uF 16V -> 10uF
- C43: renamed from C40; value 100uF 16V -> 100uF; footprint Capacitor_SMD:C_1210_3225Metric -> Capacitor_SMD:CP_Elec_6.3x5.2; moved to F.Cu
- C45: renamed from C53; value 0.1u -> 100n
- C47: renamed from C51; value 2200p -> 2.2n
- C49: renamed from C86; value 0.1u -> 100n
- C50: value 0.1u -> 100n
- C51: renamed from C34; value 0.1u -> 100n
- C52: renamed from C33; value 0.1u -> 100n
- C53: renamed from C16; value 0.1u -> 100n
- C56: renamed from C19; value 0.1u -> 100n
- C59: renamed from C81; value 0.1u -> 100n
- C60: renamed from C82; value 0.1u -> 100n
- C61: renamed from C80; value 0.1u -> 100n
- C62: renamed from C84; value 0.1u -> 100n
- C63: renamed from C85; value 0.1u -> 100n
- C64: renamed from C69; value 0.1u -> 100n
- C65: renamed from C70; value 0.1u -> 100n
- C66: renamed from C71; value 0.1u -> 100n
- C67: renamed from C72; value 0.1u -> 100n
- C68: renamed from C73; value 0.1u -> 100n
- C69: renamed from C74; value 0.1u -> 100n
- C70: renamed from C75; value 0.1u -> 100n
- C71: renamed from C76; value 0.1u -> 100n
- C72: renamed from C77; value 0.1u -> 100n
- C73: renamed from C88; value 10uF 16V -> 10uF
- C74: renamed from C87; value 10uF 16V -> 10uF
- C9: renamed from C3; value 0.01u -> 10n
- R45: renamed from R13; value 39.0K 1% -> 39K
- R46: renamed from R14; value 100.0K 1% -> 100K
- moved C43 9.40 mm to (181.4, 87.6)
- moved C32 5.03 mm to (179.8, 80.4)
- moved R36 2.86 mm to (187.3, 98.9)
- moved C36 2.41 mm to (185.4, 76.8), turned to -90 degrees
- moved REF** 2.24 mm to (181.2, 68.0)
- moved C33 2.01 mm to (182.1, 94.9)
- moved R37 1.67 mm to (186.0, 82.4), turned to 90 degrees
- moved G1 0.15 mm to (135.3, 83.2)
- moved C45 0.13 mm to (150.3, 61.8), turned to -90 degrees
- renumbered C62 to C1, C61 to C2, C55 to C24, C79 to C3, C30 to C36, C32 to C37, C64 to C4, C41 to C40, C59 to C44, C52 to C46, C35 to C48, C68 to C5, C100 to C54, C44 to C55, C101 to C57, C45 to C58, C67 to C6, C65 to C7, C66 to C8, J2 to CN1, J4 to CN2, J6 to CN3, J3 to J1, IO1 to JP1, J5 to JP2, JP1 to JP3, JP2 to JP4, J7 to JP5, T1 to Q1, T2 to Q2, R41 to R1, R4 to R10, R21 to R11, R23 to R12, R46 to R13, R47 to R14, R48 to R15, R49 to R16, R45 to R17, R1 to R18, R2 to R19, R44 to R2, R39 to R20, R35 to R21, R33 to R22, R32 to R23, R36 to R24, R37 to R25, R29 to R26, R30 to R27, R25 to R28, R22 to R29, R43 to R3, R28 to R30, R19 to R32, R20 to R33, R50 to R34, R52 to R35, R55 to R36, R56 to R37, R7 to R38, R6 to R39, R42 to R4, R5 to R40, R8 to R41, R16 to R42, R17 to R43, R15 to R44, R9 to R47, R24 to R48, R38 to R49, R53 to R5, R18 to R50, R10 to R51, R11 to R52, R12 to R53, R27 to R54, R26 to R55, R51 to R6, R40 to R7, R34 to R8, R3 to R9, J1 to SL1, U31 to U1, U14 to U11, U15 to U12, U9 to U13, U24 to U14, U17 to U15, U25 to U16, U8 to U17, U7 to U18, U2 to U19, U32 to U2, U3 to U20, U34 to U21, U33 to U22, U16 to U24, U27 to U25, U28 to U26, U20 to U27, U26 to U28, U12 to U3, U11 to U30, U5 to U31, U6 to U32, U4 to U33, U1 to U4, U30 to U5, U22 to U6, U21 to U7, U19 to U8, U18 to U9
Connections:
- C32 pad 2: Net-(C105-Pad2) -> Net-(C32-Pad2)
- C33 pad 2: Net-(C106-Pad2) -> Net-(C33-Pad2)
- C34 pad 2: Net-(C107-Pad2) -> Net-(C33-Pad2)
- C35 pad 2: Net-(C108-Pad2) -> Net-(C32-Pad2)
- C45 pad 1: -12V -> GND
- C45 pad 2: GND -> -12V
- CN2 pad R: Net-(C108-Pad2) -> Net-(C32-Pad2)
- CN2 pad T: Net-(C107-Pad2) -> Net-(C33-Pad2)
- R36 pad 2: Net-(C106-Pad2) -> Net-(C33-Pad2)
- R37 pad 2: Net-(C105-Pad2) -> Net-(C32-Pad2)
- U21 pad 14: unconnected-(U34A-VCC-Pad14) -> VCC
- U21 pad 7: unconnected-(U34A-GND-Pad7) -> GND
- U22 pad 14: unconnected-(U33A-VCC-Pad14) -> VCC
- U22 pad 7: unconnected-(U33A-GND-Pad7) -> GND
Routing:
- net Net-(C33-Pad2): track 0.00 -> 24.2 mm, vias 0 -> 1
- net Net-(C32-Pad2): track 0.00 -> 20.2 mm
- net Net-(C107-Pad2): track 14.8 -> 0.00 mm, vias 1 -> 0
- net Net-(U32A--): track 27.2 -> 40.7 mm, vias 0 -> 1
- net Net-(C43-Pad2): track 3.83 -> 14.9 mm, vias 0 -> 1
- net Net-(C108-Pad2): track 9.93 -> 0.00 mm
- net Net-(C105-Pad2): track 6.73 -> 0.00 mm
- net Net-(C106-Pad2): track 6.52 -> 0.00 mm
- net VCC: track 143.1 -> 147.8 mm, vias 36 -> 39
- net Net-(U33-OUT_A): track 14.5 -> 19.0 mm
- net GND: track 145.9 -> 149.0 mm, vias 46 -> 50
- net Net-(U33-OUT_B): track 11.9 -> 13.8 mm
- net Net-(C36-Pad1): track 9.95 -> 11.4 mm
- net +5VA: track 18.8 -> 20.0 mm
Other:
- board text added: "Designed in Romania"
- board text added: "JLCJLCJLCJLC"
- board text added: "Rev 1A"
- board text added: "by computerguy096"
