File: kicad/SnarkBarker.kicad_sch (KiCad schematic)
At the start: 194 parts, among them J1 Bus_ISA_8bit, J2 Bracket Mount, P1 Joystick/MIDI, P2 L7809, T1 2N3904, T2 2N3904, U1 NE558, U10 YM3014B, U11 NJM3403A, U12 MC1408_DIP, U13 805X, U14 SAA1099, U15 SAA1099, U16 74LS08, U17 74LS139, U18 74LS374, U19 74LS374, U2 74LS245, U20 74LS74, U21 74LS125, U22 74LS74, U23 74LS74, U24 74LS32, U25 74LS08, U26 74LS74, U27 74LS32, U28 74LS08, U29 74LS14, U3 74LS244, U30 74LS32, U4 TEA2025B, U5 LM324, U6 LM393, U7 74LS138, U8 74LS138, U9 YM3812

Commit message: finalized the migration to kicad 9
Parts:
- removed C1, C14, C42, C43, C46: 10uF 16V, SoundBlaster:SB_C_RADIAL_75_150, symbol SnarkBarker-rescue:CP1_Small
- removed C10, C47, C48, C5, C56, C6, C8, C83, C9: 0.1u, SoundBlaster:SB_C_AXIAL_275, symbol SnarkBarker-rescue:C_Small
- removed C11, C4: 470uF 16V, SoundBlaster:SB_C_RADIAL_100_320, symbol SnarkBarker-rescue:CP1_Small
- removed C12, C15, C17, C18, C3, C7: 100uF 16V, SoundBlaster:SB_C_RADIAL_100_320, symbol SnarkBarker-rescue:CP1_Small
- removed C13, C2: 47uF 16V, SoundBlaster:SB_C_RADIAL_75_150, symbol SnarkBarker-rescue:CP1_Small
- removed C20, C21, C22, C24, C25, C26, C27, C28, C29: 0.01u, SoundBlaster:SB_C_DISC_200, symbol SnarkBarker-rescue:C_Small
- removed C36, C37, C49, C54: 1000p, SoundBlaster:SB_C_DISC_200, symbol SnarkBarker-rescue:C_Small
- removed DRQ1: DMA ENABLE JUMPER, SoundBlaster:SB_HDR_1X2, symbol SnarkBarker-rescue:Jumper_NC_Small
- removed IRQ2, IRQ3, IRQ5, IRQ7: Conn_02x01, SoundBlaster:SB_HDR_1X2, symbol SnarkBarker-rescue:Conn_02x01
- removed J2: Bracket Mount, SoundBlaster:SB_MH_125, symbol SnarkBarker-rescue:Conn_01x01
- removed L1, L2, L3: BEAD, SoundBlaster:SB_L_AXIAL_500, symbol SnarkBarker-rescue:L_Core_Ferrite_Small
- removed MIC1: Microphone, SoundBlaster:SB_MJ-3536N, symbol SnarkBarker-rescue:Audio-Jack-2_Switch
- removed P1: Joystick/MIDI, SoundBlaster:SB_DB15_152-3415, symbol SnarkBarker-rescue:DB15_Female_MountingHoles
- removed P2: L7809, SoundBlaster:SB_TO220, symbol SnarkBarker-rescue:L7809
- removed R1, R2: 270, SoundBlaster:SB_R_AXIAL_400, symbol SnarkBarker-rescue:R_Small
- removed R19, R20, R21: 390, SoundBlaster:SB_R_AXIAL_400, symbol SnarkBarker-rescue:R_Small
- removed R23, R24, R3, R34, R4, R40: 10K, SoundBlaster:SB_R_AXIAL_400, symbol SnarkBarker-rescue:R_Small
- removed RP1: 2.2K, SoundBlaster:SB_RP_4B, symbol SnarkBarker-rescue:R_Pack04_SIP
- removed RP2, RP3: 1K, SoundBlaster:SB_RP_4C, symbol SnarkBarker-rescue:R_Network04
- removed RXD1, TXD1: Conn_01x03, SoundBlaster:SB_HDR_1X3, symbol SnarkBarker-rescue:Conn_01x03
- removed R_BODGE1: 4.7K, symbol SnarkBarker-rescue:R
- removed S1: OUT, SoundBlaster:SB_SJ1-3553, symbol SnarkBarker-rescue:Audio-Jack-3
- removed S2: ALPS_RK08H_DUAL, SoundBlaster:SB_ALPS_RK08_DUAL, symbol SnarkBarker-rescue:ALPS_RK08H_DUAL
- removed U10: YM3014B, SoundBlaster:SB_DIP8_300, symbol SnarkBarker-rescue:YM3014B
- removed U11: NJM3403A, SoundBlaster:SB_DIP14_300, symbol SnarkBarker-rescue:LM324
- removed U13: 805X, SoundBlaster:SB_DIP40_600, symbol SnarkBarker-rescue:805X
- removed U14, U15: SAA1099, SoundBlaster:SB_DIP18_300, symbol SnarkBarker-rescue:SAA1099
- removed U16, U25, U28: 74LS08, SoundBlaster:SB_DIP14_300, symbol SnarkBarker-rescue:74LS08
- removed U22: 74LS74, SoundBlaster:SB_DIP14_300, symbol SnarkBarker-rescue:74LS74
- removed U24, U30: 74LS32, SoundBlaster:SB_DIP14_300, symbol SnarkBarker-rescue:74LS32
- removed U3: 74LS244, SoundBlaster:SB_DIP20_300, symbol SnarkBarker-rescue:74LS244
- removed U4: TEA2025B, SoundBlaster:SB_DIP16_300, symbol SnarkBarker-rescue:TEA2025
- removed U6: LM393, SoundBlaster:SB_DIP8_300, symbol SnarkBarker-rescue:LM393
- removed U9: YM3812, SoundBlaster:SB_DIP24_600, symbol SnarkBarker-rescue:YM3812
- removed XTL1: 12MHz, SoundBlaster:SB_XTAL_HC49U_RA, symbol SnarkBarker-rescue:Crystal_GND24
- removed ZD1, ZD2, ZD3: 5.1V, SoundBlaster:SB_D_AXIAL_400_ALT, symbol SnarkBarker-rescue:D_Zener_Small_ALT
- added C100, C101: 10uF, Capacitor_SMD:C_1210_3225Metric, symbol Device:C_Polarized_Small
- added C102, C103, C104: 1µF, Capacitor_SMD:C_0805_2012Metric, symbol Device:C_Small
- added C105, C106: 100µF 25V, Capacitor_SMD:CP_Elec_6.3x5.2, symbol Device:C_Polarized
- added C107, C108: 100pF, Capacitor_SMD:C_0805_2012Metric, symbol Device:C_Small
- added C90, C93, C94, C95, C97: 150nF, Capacitor_SMD:C_0805_2012Metric, symbol Device:C_Small
- added C91, C92, C96: 22nF, Capacitor_SMD:C_0805_2012Metric, symbol Device:C_Small
- added C98, C99: 100nF, Capacitor_SMD:C_0805_2012Metric, symbol Device:C_Small
- added J2: GAME, Connector_Dsub:DSUB-15_Pins_Horizontal_P2.77x2.84mm_EdgePinOffset7.70mm_Housed_MountingHolesOffset9.12mm, symbol Connector:DA15_Pins_MountingHoles
- added J4, J6: SPKOUT, Connector_Audio:Jack_3.5mm_CUI_SJ1-3535NG_Horizontal, symbol Connector_Audio:AudioJack3_SwitchTR
- added J5: IRQ, Connector_PinHeader_2.54mm:PinHeader_2x04_P2.54mm_Vertical, symbol Connector_Generic:Conn_02x04_Odd_Even
- added JP2: DMA EN, Connector_PinHeader_2.54mm:PinHeader_1x02_P2.54mm_Vertical, symbol Connector:Conn_01x02_Pin
- added R1, R2: 10K, Resistor_SMD:R_0805_2012Metric, symbol Device:R_Small
- added R19, R20, R50, R52: 20K, Resistor_SMD:R_0805_2012Metric, symbol Device:R
- added R21, R23, R3, R34, R4, R40, R51, R53, R55, R56: 1K, Resistor_SMD:R_0805_2012Metric, symbol Device:R
- added R24: 4.7K, Resistor_SMD:R_0805_2012Metric, symbol Device:R_Small
- added R45: 47, Resistor_SMD:R_0805_2012Metric, symbol Device:R
- added R46, R47, R48, R49: 2k, Resistor_SMD:R_0805_2012Metric, symbol Device:R
- added R57, R58: 0, Resistor_SMD:R_0805_2012Metric, symbol Device:R
- added U1: AT89LP51, Package_QFP:TQFP-44_10x10mm_P0.8mm, symbol MCU_Microchip_8051:AT89x51xxA
- added U10: YM3014, Package_DIP:DIP-8_W7.62mm, symbol SB:YM3014
- added U11: LM324, Package_SO:SOIC-14_3.9x8.7mm_P1.27mm, symbol Amplifier_Operational:LM324
- added U14, U15: SAA1099, Package_DIP:DIP-18_W7.62mm, symbol SB:SAA1099
- added U16, U25, U28: 74LS08, Package_SO:SOIC-14_3.9x8.7mm_P1.27mm, symbol 74xx:74LS08
- added unit 3 of U17
- added unit 3 of U20
- added unit 5 of U21
- added U22: 74LS74, Package_SO:SOIC-14_3.9x8.7mm_P1.27mm, symbol 74xx:74LS74
- added unit 3 of U23
- added U24, U30: 74LS32, Package_SO:SOIC-14_3.9x8.7mm_P1.27mm, symbol 74xx:74LS32
- added unit 3 of U26
- added unit 5 of U27
- added unit 7 of U29
- added U3: 74LS245, Package_SO:SOIC-20W_7.5x12.8mm_P1.27mm, symbol 74xx:74LS245
- added U31: L7805, Package_TO_SOT_THT:TO-220-3_Horizontal_TabDown, symbol Regulator_Linear:L7805
- added U32: L7905, Package_TO_SOT_THT:TO-220-3_Horizontal_TabDown, symbol Regulator_Linear:L7905
- added U4: LM4880MX, Package_SO:SO-8_3.9x4.9mm_P1.27mm, symbol SB:LM4880MX
- added unit 5 of U5
- added U6: LM393, Package_SO:SOIC-8_3.9x4.9mm_P1.27mm, symbol Comparator:LM393
- added U9: YM3812, Package_DIP:DIP-24_W15.24mm, symbol SB:YM3812
- added Y1: 12MHz, Crystal:Crystal_HC49-U_Vertical, symbol Device:Crystal
- C16, C19, C33, C34, C50, C53, C69, C70, C71, C72, C73, C74, C75, C76, C77, C80, C81, C82, C84, C85, C86, C89: footprint SoundBlaster:SB_C_AXIAL_275 -> Capacitor_SMD:C_0805_2012Metric; symbol SnarkBarker-rescue:C_Small -> Device:C_Small
- C23, C31, C32, C35, C41, C51, C52, C57, C58, C59, C60, C61, C62, C63, C64, C65, C66, C67, C68, C78, C79: footprint SoundBlaster:SB_C_DISC_200 -> Capacitor_SMD:C_0805_2012Metric; symbol SnarkBarker-rescue:C_Small -> Device:C_Small
- C30, C38, C39, C87, C88: footprint SoundBlaster:SB_C_RADIAL_75_150 -> Capacitor_SMD:C_1210_3225Metric; symbol SnarkBarker-rescue:CP1_Small -> Device:C_Polarized_Small
- C40: footprint SoundBlaster:SB_C_RADIAL_100_320 -> Capacitor_SMD:C_1210_3225Metric; symbol SnarkBarker-rescue:CP1_Small -> Device:C_Polarized_Small
- C44, C45, C55: value 10uF 16V -> 10uF; footprint SoundBlaster:SB_C_RADIAL_75_150 -> Capacitor_SMD:C_1210_3225Metric; symbol SnarkBarker-rescue:CP1_Small -> Device:C_Polarized_Small
- D1, D2: footprint SoundBlaster:SB_D_AXIAL_400 -> Diode_SMD:D_0805_2012Metric; symbol SnarkBarker-rescue:D_Small_ALT -> Diode:1N4148
- IO1: footprint SoundBlaster:SB_HDR_2X6 -> Connector_PinHeader_2.54mm:PinHeader_2x06_P2.54mm_Vertical; symbol SnarkBarker-rescue:Conn_02x06_Odd_Even -> Connector_Generic:Conn_02x06_Odd_Even
- J1: value Bus_ISA_8bit -> 8-bit ISA slot; footprint SoundBlaster:BUS_PC -> SB:ISA card edge; symbol SnarkBarker-rescue:Bus_ISA_8bit -> Connector:Bus_ISA_8bit
- JP1: footprint SoundBlaster:SB_HDR_1X2 -> Connector_PinHeader_2.54mm:PinHeader_1x02_P2.54mm_Vertical; symbol SnarkBarker-rescue:Jumper_NC_Small -> Connector:Conn_01x02_Pin
- R10, R11, R12, R13, R14, R15, R16, R17, R22, R25, R26, R27, R28, R29, R30, R31, R32, R33, R35, R36, R37, R39, R41, R42, R43, R44, R5, R6, R7, R8, R9: footprint SoundBlaster:SB_R_AXIAL_400 -> Resistor_SMD:R_0805_2012Metric; symbol SnarkBarker-rescue:R_Small -> Device:R_Small
- R18: value 1.5K 1% -> 1.5K; footprint SoundBlaster:SB_R_AXIAL_400 -> Resistor_SMD:R_0805_2012Metric; symbol SnarkBarker-rescue:R_Small -> Device:R_Small
- R38: value 2.70K 1% -> 2.7K; footprint SoundBlaster:SB_R_AXIAL_400 -> Resistor_SMD:R_0805_2012Metric; symbol SnarkBarker-rescue:R_Small -> Device:R_Small
- T1, T2: footprint SoundBlaster:SB_TO92 -> Package_TO_SOT_SMD:SOT-23; symbol SnarkBarker-rescue:2N3904 -> Transistor_BJT:2N3904
- U12: value MC1408_DIP -> MC1408; footprint SoundBlaster:SB_DIP16_300 -> Package_SO:SOIC-16_3.9x9.9mm_P1.27mm; symbol SnarkBarker-rescue:MC1408-8_DIP -> Analog_DAC:MC1408_SOIC
- U13: renamed from U1; footprint SoundBlaster:SB_DIP16_300 -> Package_SO:SOIC-16_4.55x10.3mm_P1.27mm; symbol SnarkBarker-rescue:NE558 -> SB:NE558
- U17: footprint SoundBlaster:SB_DIP16_300 -> Package_SO:SOIC-16_3.9x9.9mm_P1.27mm; symbol SnarkBarker-rescue:74LS139 -> 74xx:74LS139
- U18, U19: footprint SoundBlaster:SB_DIP20_300 -> Package_SO:SOIC-20W_7.5x12.8mm_P1.27mm; symbol SnarkBarker-rescue:74LS374 -> 74xx:74LS374
- U2: footprint SoundBlaster:SB_DIP20_300 -> Package_SO:SOIC-20W_7.5x12.8mm_P1.27mm; symbol SnarkBarker-rescue:74LS245 -> 74xx:74LS245
- U20, U23, U26: footprint SoundBlaster:SB_DIP14_300 -> Package_SO:SOIC-14_3.9x8.7mm_P1.27mm; symbol SnarkBarker-rescue:74LS74 -> 74xx:74LS74
- U21: footprint SoundBlaster:SB_DIP14_300 -> Package_SO:SOIC-14_3.9x8.7mm_P1.27mm; symbol SnarkBarker-rescue:74LS125 -> 74xx:74LS125
- U27: footprint SoundBlaster:SB_DIP14_300 -> Package_SO:SOIC-14_3.9x8.7mm_P1.27mm; symbol SnarkBarker-rescue:74LS32 -> 74xx:74LS32
- U29: footprint SoundBlaster:SB_DIP14_300 -> Package_SO:SOIC-14_3.9x8.7mm_P1.27mm; symbol SnarkBarker-rescue:74LS14 -> 74xx:74LS14
- U5: footprint SoundBlaster:SB_DIP14_300 -> Package_SO:SOIC-14_3.9x8.7mm_P1.27mm; symbol SnarkBarker-rescue:LM324 -> Amplifier_Operational:LM324; Mouser 595-LM324AN -> 512-LM324AN
- U5: footprint SoundBlaster:SB_DIP14_300 -> Package_SO:SOIC-14_3.9x8.7mm_P1.27mm; symbol SnarkBarker-rescue:LM324 -> Amplifier_Operational:LM324
- U7, U8: footprint SoundBlaster:SB_DIP16_300 -> Package_SO:SOIC-16_3.9x9.9mm_P1.27mm; symbol SnarkBarker-rescue:74LS138 -> 74xx:74LS138
Connections:
- net +12V: now also C101.1, U31.1 (IN); no longer C16.1
- net +5VA: now also R24.1, U11.4 (V+), U31.3 (OUT), U4.8 (VDD), U5.4 (V+), U6.8 (V+); no longer U5.4 (V+)
- net -12V: now also C16.1, U12.7 (VEE), C100.2, U32.2 (VI); no longer U12.3 (VEE)
- net A0: now also U14.3 (A0), U15.3 (A0), U9.4 (A0)
- net A3: now also U24.2
- net D0: now also U14.10 (D0), U15.10 (D0), U3.2 (A0), U9.10 (D0)
- net D1: now also U14.11 (D1), U15.11 (D1), U3.3 (A1), U9.11 (D1)
- net D2: now also U14.12 (D2), U15.12 (D2), U3.4 (A2), U9.13 (D2)
- net D3: now also U14.13 (D3), U15.13 (D3), U3.5 (A3), U9.14 (D3)
- net D4: now also U14.14 (D4), U15.14 (D4), U3.6 (A4), U9.15 (D4)
- net D5: now also U14.15 (D5), U15.15 (D5), U3.7 (A5), U9.16 (D5)
- net D6: now also U14.16 (D6), U15.16 (D6), U3.8 (A6), U9.17 (D6)
- net D7: now also U14.17 (D7), U15.17 (D7), U3.9 (A7), U9.18 (D7)
- net DAC0: now also U12.9 (A1), U1.40 (P1.0); no longer U12.12 (A1)
- net DAC1: now also U12.10 (A2), U1.41 (P1.1); no longer U12.11 (A2)
- net DAC2: now also U12.11 (A3), U1.42 (P1.2); no longer U12.10 (A3)
- net DAC3: now also U12.12 (A4), U1.43 (P1.3); no longer U12.9 (A4)
- net DAC4: now also U12.13 (A5), U1.44 (P1.4); no longer U12.8 (A5)
- net DAC5: now also U12.14 (A6), U1.1 (P1.5); no longer U12.7 (A6)
- net DAC6: now also U12.15 (A7), U1.2 (P1.6); no longer U12.6 (A7)
- net DAC7: now also U12.16 (A8), U1.3 (P1.7/SCK); no longer U12.5 (A8)
- net DAV_DSP: now also U1.25 (P2.7/A15), U22.9 (Q), U30.10
- net DAV_PC: now also U1.24 (P2.6/A14), U22.5 (Q)
- net DD0: now also U1.37 (P0.0/AD0)
- net DD1: now also U1.36 (P0.1/AD1)
- net DD2: now also U1.35 (P0.2/AD2)
- net DD3: now also U1.34 (P0.3/AD3)
- net DD4: now also U1.33 (P0.4/AD4)
- net DD5: now also U1.32 (P0.5/AD5)
- net DD6: now also U1.31 (P0.6/AD6)
- net DD7: now also U1.30 (P0.7/AD7)
- net DREQUEST: now also U1.11 (P3.5)
- net DRQ1: now also JP2.2 (Pin_2)
- net DSPRD_~{CS}: now also U28.10
- net DSPRST_~{CS}: now also U24.13
- net DSPWR_~{CS}: now also U28.13
- net DSP_BUSY: now also U1.9 (P3.3), U30.9
- net FM_~{CS}: now also U9.7 (~{CS})
- net GND: now also C16.2, C19.2, C23.1, C32.1, C33.2, C34.2, C35.2, C39.2, C44.1, C45.2, C50.2, C52.1, C53.2, C55.2, C57.2, C58.2, C60.2, C61.1, C62.1, C63.2, C78.2, C81.2, C82.2, C86.2, C87.2, C89.2, D1.2 (A), J1.1 (GND), R12.2, R13.2, R5.2, T1.1 (E), T2.1 (E), U12.3 (VREF-), U12.6 (GND), U13.12 (GND), U5.10 (+), C100.1, C101.2, C104.1, C107.1, C108.1, C90.1, C91.1, C92.1, C93.1, C94.1, C95.1, C96.1, C97.1, C98.1, C99.1, J2.0 (PAD), J2.4, J2.5, J4.S, J6.S, R55.1, R56.1, U1.16 (GND), U1.17 (GND), U10.6 (GND), U14.9 (VSS), U15.9 (VSS), U16.7 (GND), U17.8 (GND), U20.7 (GND), U21.7 (GND), U22.12 (D), U22.2 (D), U22.7 (GND), U23.7 (GND), U24.7 (GND), U25.7 (GND), U26.7 (GND), U27.7 (GND), U28.7 (GND), U29.7 (GND), U3.1 (A->B), U3.10 (GND), U30.7 (GND), U31.2 (GND), U32.1 (GND), U4.4 (GND), U4.5 (SHUTDOWN), U5.11 (V-), U6.4 (V-), U6.5 (+), U6.6 (-), U9.12 (GND); no longer C61.2, C62.2, U17.8 (GND), U17.8 (GND), U20.7 (GND), U20.7 (GND), U21.7 (GND), U21.7 (GND), U21.7 (GND), U21.7 (GND), U23.7 (GND), U23.7 (GND), U26.7 (GND), U26.7 (GND), U27.7 (GND), U27.7 (GND), U27.7 (GND), U27.7 (GND), U29.7 (GND), U29.7 (GND), U29.7 (GND), U29.7 (GND), U29.7 (GND), U29.7 (GND)
- net IREQUEST: now also U1.8 (P3.2)
- net IRQ2: now also J5.8 (Pin_8)
- net IRQ3: now also J5.6 (Pin_6)
- net IRQ5: now also J5.4 (Pin_4)
- net IRQ7: now also J5.2 (Pin_2)
- net MIC_COMP: now also U1.23 (P2.5/A13), U6.1
- net MIDI_IN: now also J2.15 (P15), U1.5 (P3.0)
- net MIDI_OUT: now also J2.12 (P12), U1.7 (P3.1)
- net MUTE_EN: now also U1.18 (P2.0/A8)
- net RESET: now also U1.4 (RST), U30.3
- net VCC: now also C81.1, C82.1, C87.1, J1.3 (VCC), R14.1, R32.2, R33.2, R38.2, R39.2, U12.1 (VCC), U13.5 (VCC), R1.2, R2.2, R21.2, R23.2, R3.2, R34.1, R4.2, R40.1, R45.1, R51.1, R53.1, U1.29 (~{EA}/V_{pp}), U1.38 (V_{cc}), U10.1 (VCC), U14.18 (VDD), U15.18 (VDD), U16.14 (VCC), U17.16 (VCC), U20.14 (VCC), U21.14 (VCC), U22.14 (VCC), U23.14 (VCC), U24.14 (VCC), U25.14 (VCC), U26.14 (VCC), U27.14 (VCC), U28.14 (VCC), U29.14 (VCC), U3.20 (VCC), U30.14 (VCC), U9.1 (VCC); no longer U17.16 (VCC), U17.16 (VCC), U20.14 (VCC), U20.14 (VCC), U21.14 (VCC), U21.14 (VCC), U21.14 (VCC), U21.14 (VCC), U23.14 (VCC), U23.14 (VCC), U26.14 (VCC), U26.14 (VCC), U27.14 (VCC), U27.14 (VCC), U27.14 (VCC), U27.14 (VCC), U29.14 (VCC), U29.14 (VCC), U29.14 (VCC), U29.14 (VCC), U29.14 (VCC), U29.14 (VCC)
- net ~{DACK1}: now also U30.5
- net ~{DB_EN}: now also U16.8
- net ~{DMAOUT}: now also U25.1, U28.12, U28.5, U28.9, U30.6
- net ~{DMA_EN}: now also U1.10 (P3.4), U30.4
- net ~{DSP_READ}: now also U1.13 (P3.7), U22.13 (~{R})
- net ~{DSP_WRITE}: now also U1.12 (P3.6), U22.4 (~{S})
- net ~{IC}: now also U25.10, U9.3 (~{IC})
- net ~{IOR}: now also U25.5
- net ~{IOW}: now also U16.5
- net ~{ISA_RD}: now also U22.1 (~{R})
- net ~{ISA_WR}: now also U22.10 (~{S})
- net ~{RD_DAV}: now also U28.1
- net ~{RD}: now also U24.10, U25.6, U9.6 (~{RD})
- net ~{RESET}: now also U22.11 (C), U22.3 (C), U28.2, U28.4
- net ~{WR}: now also U14.1 (~{WR}), U15.1 (~{WR}), U16.6, U24.12, U24.4, U9.5 (~{WR})
- net RB: now reaches C55.1
- net RB: now also U10.7 (RB), U11.3 (+)
- net at U13.1 (OUTPUT_A): now also R40.2, U3.15 (B3)
- net GAME_ANALOG2: now reaches U13.10 (TIMING_C)
- net GAME_ANALOG2: now also C95.2, R46.1
- net at U13.11 (TRIGGER_C), U13.14 (TRIGGER_D), U13.3 (TRIGGER_A)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: now also U24.6
- net GAME_ANALOG1: now reaches U13.15 (TIMING_D)
- net GAME_ANALOG1: now also C92.2, R49.1
- net at U13.16 (OUTPUT_D): now also R34.2, U3.18 (B0)
- net GAME_ANALOG4: now reaches U13.2 (TIMING_A)
- net GAME_ANALOG4: now also C91.2, R47.1
- net at U13.4 (CV): now also C23.2; no longer C23.1
- net GAME_ANALOG3: now reaches U13.7 (TIMING_B)
- net GAME_ANALOG3: now also C96.2, R48.1
- net at U13.8 (OUTPUT_B): now also R51.2, U3.16 (B2)
- net at U13.9 (OUTPUT_C): now also R53.2, U3.17 (B1)
- net at R10.2, R18.2, U5.8: now also U6.3 (+)
- net at R18.1, U5.9 (-): now also U12.8 (I0); no longer U12.4 (I0)
- net at C40.1, C41.1, R9.1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: now also R24.2, U6.2 (-)
- net IO250: now reaches IO1.9 (Pin_9), U7.10 (O5)
- net IO240: now reaches IO1.7 (Pin_7), U7.11 (O4)
- net IO230: now reaches IO1.5 (Pin_5), U7.12 (O3)
- net IO220: now reaches IO1.3 (Pin_3), U7.13 (O2)
- net IO210: now reaches IO1.1 (Pin_1), U7.14 (O1)
- net IO260: now reaches IO1.11 (Pin_11), U7.9 (O6)
- net at R22.1, R30.1, R31.1: now also C103.1
- net at R25.1, R28.1, R29.1: now also C102.1
- net at R35.2: now also U11.6 (-), U11.7
- net at R38.1: now also U12.2 (VREF+); no longer U12.14 (VREF+)
- net at C59.1: now also U12.4 (COMPEN); no longer U12.16 (COMPEN)
- net OUTR: now reaches C63.1, R36.2
- net OUTR: now also R33.1, U14.4 (OUTR), U15.4 (OUTR); no longer R32.1
- net OUTL: now reaches C78.1, R37.2
- net OUTL: now also R32.1, U14.5 (OUTL), U15.5 (OUTL); no longer R33.1
- net at R41.2: now also U16.4
- net at U20.1 (~{R}): now also U28.6
- net at U20.10 (~{S}): now also U25.8
- net at U20.12 (D): now also U25.11
- net at U21.5: now also U30.8
- net at C65.1, R43.1, U21.11: now also JP2.1 (Pin_1)
- net at JP1.1 (Pin_1): now also U24.3
- net at U26.3 (C): now also U24.11
- net at R44.2: now also U25.4
- net at U26.5 (Q): now also U30.1
- net at U26.13 (~{R}): now also U28.3
- net at U26.9 (Q): now also J5.1 (Pin_1), J5.3 (Pin_3), J5.5 (Pin_5), J5.7 (Pin_7)
- net at U27.1: now also U28.8
- net at U27.10: now also U28.11
- net at C30.2: now also J6.R
- removed net +5VD: R14.1, R32.2, R33.2, R38.2, R39.1
- net +9VA renamed -5V
- net -5V: now also C33.1, C44.2, C50.1, U11.11 (V-), U32.3 (VO)
- removed net -5VA: C33.1, C44.2, C50.1, U5.11 (V-)
- net 1xx000xxxx: no longer names the net of U17.1 (E), U7.15 (O0)
- net BUSRESET renamed RST
- net RST: now also U30.2
- net CLK_14M318 renamed CLK
- net CLK_3M579 renamed CLK/4
- net CLK/4: now also U9.24 (PM)
- net CLK_7M159 renamed CLK/2
- net CLK/2: now also U14.8 (CLK), U15.8 (CLK)
- net CMS1-6_~{CS} renamed CMS0
- net CMS0: now also U15.2 (~{CS}), U25.12
- net CMS7-12_~{CS} renamed CMS1
- net CMS1: now also U14.2 (~{CS}), U25.13
- net DIGITAL_OUT renamed DSPOUT
- removed net GNDA: C16.2, C19.2, C23.2, C32.1, C33.2, C34.2, C35.2, C39.2, C44.1, C45.2, C50.2, C52.1, C53.2, C55.2, C57.2, C58.2, C60.2, C63.2, C78.2, C81.2, C82.2, C86.2, C87.2, C89.2, D1.2 (A), J1.1 (GND), R12.2, R13.2, R5.2, T1.1 (E), T2.1 (E), U12.1 (NC), U12.15 (VREF-), U12.2 (GND), U13.12 (GND), U5.10 (+)
- net IO_READY renamed IORDY
- net JOYSTICK_~{CS} renamed ~{JOYCS}
- net ~{JOYCS}: now also U24.5, U24.9, U25.2
- net OPL2 renamed FMOUT
- net SAA_L: no longer names the net of C60.1, R30.2, R37.1
- net SAA_R: no longer names the net of C58.1, R29.2, R36.1
- removed net VDDA: C81.1, C82.1, C87.1, J1.3 (VCC), U12.13 (VCC), U13.5 (VCC)
- net ~{100000xxxx}: no longer names the net of U17.4 (O0)
- net ~{100000xxxx}: now also U24.1
- net ~{100jjjxxxx}: no longer names the net of U17.12 (O0)
- net ~{100jjjxxxx}: now also U16.2
- net ~{111000xxxx}: no longer names the net of U17.7 (O3)
- net ~{111000xxxx}: now also U16.1
- net ~{CARD_SELECTED} renamed ~{CS}
- net ~{CS}: now also U16.3, U16.9
- new net: C61.2, U1.14 (XTAL2), Y1.2
- new net: C62.2, U1.15 (XTAL1), Y1.1
- new net: U16.10, U25.3
- new net: C107.2, J4.T, R58.1
- new net: C105.1, R50.2, U4.1 (OUT_A)
- new net: R19.2, R50.1, U4.2 (IN_A)
- new net: C104.2, U4.3 (BYPASS)
- new net: R20.2, R52.1, U4.6 (IN_B)
- new net: C106.1, R52.2, U4.7 (OUT_B)
- new net: U24.8, U3.19 (CE)
- new net: C103.2, R20.1
- new net: R1.1, U14.6 (IREF)
- new net: C108.2, J4.R, R57.1
- new net: R2.1, U15.6 (IREF)
- new net: J2.13 (P13), R47.2
- new net: J2.11 (P111), R48.2
- new net: C105.2, R56.2, R57.2
- new net: C102.2, R19.1
- new net: C106.2, R55.2, R58.2
- new net: U10.2 (BUFF), U11.5 (+)
- new net: U9.19 (NC), U9.22 (NC), U9.8 (NC), U9.9 (NC)
- new net: U10.3 (LOAD), U9.20 (SH)
- new net: U10.4 (SD), U9.21 (MO)
- new net: U10.5 (CLOCK), U9.23 (SY)
- new net: J2.3, R49.2
- new net: J2.6, R46.2
- new net DTACK: R39.1, U14.7 (~{DTACK}), U15.7 (~{DTACK}), U25.9
- new net GAME_5V: C98.2, C99.2, J2.1, J2.8, J2.9 (P9), R45.2
- new net GAME_DIGITAL1: C93.2, J2.2, R3.1, U3.14 (B4)
- new net GAME_DIGITAL2: C94.2, J2.7, R4.1, U3.13 (B5)
- new net GAME_DIGITAL3: C97.2, J2.10 (P10), R21.1, U3.12 (B6)
- new net GAME_DIGITAL4: C90.2, J2.14 (P14), R23.1, U3.11 (B7)
- new net MP: U10.8 (MP), U11.1, U11.2 (-)
- no-connect marks 60 -> 70
Other:
- note added: "CMS MUSIC CHIPS"
- note added: "JOYSTICK"
- note removed: "210 220 230 240 250 260"
- note removed: "8-BIT ISA BUS"
- note removed: "ADDRESS DECODERS"
- note removed: "BIDIRECTIONAL DSP BUS LATCH"
- note removed: "BYPASS CAPS"
- note removed: "COMPARATOR"
- note removed: "CREATIVE CMS MUSIC CHIPS"
- note removed: "DATA AVAILABLE FOR DSP (FLAG)"
- note removed: "DATA AVAILABLE FOR PC (FLAG)"
- note removed: "DATA AVAILABLE FROM DSP (2xEh, read)"
- note removed: "DIGITAL SOUND PROCESSOR"
- note removed: "EMI FILTERS"
- note removed: "ISA DATA BUS BUFFER"
- note removed: "JOYSTICK CIRCUIT"
- note removed: "LEFT"
- note removed: "LOW NOISE POWER SUPPLIES"
- note removed: "MIXER"
- note removed: "PULSE LOW TO CLEAR INTERRUPT"
- note removed: "RESET REGISTER (2x6h, write)"
- note removed: "REVERSED BY @TubeTimeUS WITH HELP FROM @GoodTofuFriday"
- note removed: "RIGHT"
- note removed: "SJ1-3553"
- note removed: "SNARK BARKER"
- note removed: "This work is licensed under the Creative Commons Attribution-ShareAlike 4.0 International License. To view a copy of this license, visit http://creativecommons.org/licenses/by-sa/4.0/ or send a letter to Creative Commons, PO Box 1866, Mountain View, CA 94042, USA."
- note removed: "VOLUME CONTROL"
- note removed: "WIRE BRIDGE"
- note removed: "WRITE BUFFER STATUS (2xCh, read)"
- title: (none) -> Snark Barker Mini
- moved on the sheet: C16, C19, C23, C31, C32, C33, C34, C35, C41, C50, C51, C52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

Commit message: routing
Parts:
- removed U12: MC1408, Package_SO:SOIC-16_3.9x9.9mm_P1.27mm, symbol Analog_DAC:MC1408_SOIC
- removed U13: NE558, Package_SO:SOIC-16_4.55x10.3mm_P1.27mm, symbol SB:NE558
- added C1, C2, C3: 0.01u, Capacitor_SMD:C_0805_2012Metric, symbol Device:C_Small
- added U12: DAC0808, Package_SO:SOIC-16_3.9x9.9mm_P1.27mm, symbol Analog_DAC:DAC0808_SOIC
- added U33, U34: NE556, Package_SO:SOIC-14_3.9x8.7mm_P1.27mm, symbol Timer:NE556
- C30: value 10uF 16V -> 10uF
- JP1: value JOYSTICK EN -> Gameport enable
- JP2: value DMA EN -> DMA Enable
Connections:
- net -12V: now also U12.7 (VEE)
- net DAC0: now also U12.9 (A1)
- net DAC1: now also U12.10 (A2)
- net DAC2: now also U12.11 (A3)
- net DAC3: now also U12.12 (A4)
- net DAC4: now also U12.13 (A5)
- net DAC5: now also U12.14 (A6)
- net DAC6: now also U12.15 (A7)
- net DAC7: now also U12.16 (A8)
- net GAME_ANALOG1: now also U34.12 (THR), U34.13 (DIS)
- net GAME_ANALOG2: now also U33.12 (THR), U33.13 (DIS)
- net GAME_ANALOG3: now also U34.1 (DIS), U34.2 (THR)
- net GAME_ANALOG4: now also U33.1 (DIS), U33.2 (THR)
- net GND: now also C1.1, C2.1, C3.1, U12.3 (VREF-), U12.6 (GND)
- net VCC: now also U12.1 (VCC)
- net ~{IC}: now also U33.10 (R), U33.4 (R), U34.10 (R), U34.4 (R)
- net TMOUT3: now reaches R40.2
- net TMOUT3: now also U3.16 (B2), U34.5 (Q); no longer U3.15 (B3)
- net JOYTMR: now reaches U24.6
- net JOYTMR: now also U33.6 (TR), U33.8 (TR), U34.6 (TR), U34.8 (TR)
- net TMOUT1: now reaches U3.18 (B0)
- net TMOUT1: now also R53.2, U34.9 (Q); no longer R34.2
- net at C23.2: now also U33.3 (CV)
- net TMOUT2: now reaches R51.2
- net TMOUT2: now also U3.17 (B1), U33.9 (Q); no longer U3.16 (B2)
- net at R18.1, U5.9 (-): now also U12.8 (I0)
- net at R38.1: now also U12.2 (VREF+)
- net at C59.1: now also U12.4 (COMPEN)
- net at C30.2, J6.R: now also J6.T
- new net: C2.2, U34.11 (CV)
- new net: C1.2, U33.11 (CV)
- new net: C3.2, U34.3 (CV)
- new net TMOUT4: R34.2, U3.15 (B3), U33.5 (Q)
- no-connect marks 70 -> 69
Other:
- moved on the sheet: C23, R34, R40, R51, R53, U24B

Commit message: routing almost finished
Parts:
- J4: footprint Connector_Audio:Jack_3.5mm_CUI_SJ1-3535NG_Horizontal -> SB:TRS jack
- J6: value SPKOUT -> MIC; footprint Connector_Audio:Jack_3.5mm_CUI_SJ1-3535NG_Horizontal -> SB:TRS jack
Connections:
- net +5VA: now also R14.1
- net -5V: now also U5.11 (V-)
- net GND: no longer U5.11 (V-)
- net VCC: no longer R14.1
Other:
- moved on the sheet: C33, C34, U5E

Commit message: finalized routing
Parts:
- added J3: Prog, Connector_PinHeader_2.54mm:PinHeader_1x07_P2.54mm_Vertical, symbol Connector:Conn_01x07_Pin
- added J7: DSP PWR, Connector_PinHeader_2.54mm:PinHeader_1x02_P2.54mm_Vertical, symbol Connector:Conn_01x02_Pin
Connections:
- net DAC4: now also J3.6 (Pin_6)
- net DAC5: now also J3.5 (Pin_5)
- net DAC6: now also J3.4 (Pin_4)
- net DAC7: now also J3.3 (Pin_3)
- net GND: now also J3.7 (Pin_7)
- net RESET: now also J3.2 (Pin_2)
- net VCC: now also J7.2 (Pin_2); no longer U1.29 (~{EA}/V_{pp}), U1.38 (V_{cc})
- new net VPP: J3.1 (Pin_1), J7.1 (Pin_1), U1.29 (~{EA}/V_{pp}), U1.38 (V_{cc})

Commit message: finalized first revision
Parts:
- removed R57, R58: 0, Resistor_SMD:R_0805_2012Metric, symbol Device:R
- added C75: 10uF, Capacitor_SMD:C_1210_3225Metric, symbol Device:C_Polarized_Small
- C10: renamed from C23; value 0.01u -> 10n
- C11: renamed from C1; value 0.01u -> 10n
- C12: renamed from C2; value 0.01u -> 10n
- C13: renamed from C94; value 150nF -> 100n
- C14: renamed from C90; value 150nF -> 100n
- C15: renamed from C95; value 150nF -> 100n
- C16: renamed from C91; value 22nF -> 22n
- C17: renamed from C96; value 22nF -> 22n
- C18: renamed from C92; value 22nF -> 22n
- C19: renamed from C97; value 150nF -> 100n
- C20: renamed from C93; value 150nF -> 100n
- C21: renamed from C98; value 100nF -> 100n
- C22: renamed from C99; value 100nF -> 100n
- C23: renamed from C57; value 4700p -> 4.7n
- C25: renamed from C63; value 1000p -> 1n
- C26: renamed from C78; value 1000p -> 1n
- C27: renamed from C58; value 2200p -> 2.2n
- C28: renamed from C60; value 2200p -> 2.2n
- C29: renamed from C102; value 1µF -> 1uF
- C30: renamed from C103; value 1µF -> 1uF
- C31: renamed from C104; value 1µF -> 1uF
- C32: renamed from C105; value 100µF 25V -> 100uF
- C33: renamed from C106; value 100µF 25V -> 100uF
- C34: renamed from C107; value 100pF -> 100p
- C35: renamed from C108; value 100pF -> 100p
- C38: renamed from C31; value 1000p -> 1n
- C39: renamed from C38; value 10uF 16V -> 10uF
- C41: renamed from C89; value 0.1u -> 100n
- C42: renamed from C39; value 10uF 16V -> 10uF
- C43: renamed from C40; value 100uF 16V -> 100uF; footprint Capacitor_SMD:C_1210_3225Metric -> Capacitor_SMD:CP_Elec_6.3x5.2
- C45: renamed from C53; value 0.1u -> 100n
- C47: renamed from C51; value 2200p -> 2.2n
- C49: renamed from C86; value 0.1u -> 100n
- C50: value 0.1u -> 100n
- C51: renamed from C34; value 0.1u -> 100n
- C52: renamed from C33; value 0.1u -> 100n
- C53: renamed from C16; value 0.1u -> 100n
- C56: renamed from C19; value 0.1u -> 100n
- C59: renamed from C81; value 0.1u -> 100n
- C60: renamed from C82; value 0.1u -> 100n
- C61: renamed from C80; value 0.1u -> 100n
- C62: renamed from C84; value 0.1u -> 100n
- C63: renamed from C85; value 0.1u -> 100n
- C64: renamed from C69; value 0.1u -> 100n
- C65: renamed from C70; value 0.1u -> 100n
- C66: renamed from C71; value 0.1u -> 100n
- C67: renamed from C72; value 0.1u -> 100n
- C68: renamed from C73; value 0.1u -> 100n
- C69: renamed from C74; value 0.1u -> 100n
- C70: renamed from C75; value 0.1u -> 100n
- C71: renamed from C76; value 0.1u -> 100n
- C72: renamed from C77; value 0.1u -> 100n
- C73: renamed from C88; value 10uF 16V -> 10uF
- C74: renamed from C87; value 10uF 16V -> 10uF
- C9: renamed from C3; value 0.01u -> 10n
- R45: renamed from R13; value 39.0K 1% -> 39K
- R46: renamed from R14; value 100.0K 1% -> 100K
- renumbered C62 to C1, C61 to C2, C55 to C24, C79 to C3, C30 to C36, C32 to C37, C64 to C4, C41 to C40, C59 to C44, C52 to C46, C35 to C48, C68 to C5, C100 to C54, C44 to C55, C101 to C57, C45 to C58, C67 to C6, C65 to C7, C66 to C8, J2 to CN1, J4 to CN2, J6 to CN3, J3 to J1, IO1 to JP1, J5 to JP2, JP1 to JP3, JP2 to JP4, J7 to JP5, T1 to Q1, T2 to Q2, R41 to R1, R4 to R10, R21 to R11, R23 to R12, R46 to R13, R47 to R14, R48 to R15, R49 to R16, R45 to R17, R1 to R18, R2 to R19, R44 to R2, R39 to R20, R35 to R21, R33 to R22, R32 to R23, R36 to R24, R37 to R25, R29 to R26, R30 to R27, R25 to R28, R22 to R29, R43 to R3, R28 to R30, R19 to R32, R20 to R33, R50 to R34, R52 to R35, R55 to R36, R56 to R37, R7 to R38, R6 to R39, R42 to R4, R5 to R40, R8 to R41, R16 to R42, R17 to R43, R15 to R44, R9 to R47, R24 to R48, R38 to R49, R53 to R5, R18 to R50, R10 to R51, R11 to R52, R12 to R53, R27 to R54, R26 to R55, R51 to R6, R40 to R7, R34 to R8, R3 to R9, J1 to SL1, U31 to U1, U14 to U11, U15 to U12, U9 to U13, U24 to U14, U17 to U15, U25 to U16, U8 to U17, U7 to U18, U2 to U19, U32 to U2, U3 to U20, U34 to U21, U33 to U22, U16 to U24, U27 to U25, U28 to U26, U20 to U27, U26 to U28, U12 to U3, U11 to U30, U5 to U31, U6 to U32, U4 to U33, U1 to U4, U30 to U5, U22 to U6, U21 to U7, U19 to U8, U18 to U9
Connections:
- net -12V: now also C45.2; no longer C45.1
- net GND: now also C45.1, U21.7 (GND), U21.7 (GND), U22.7 (GND), U22.7 (GND), C75.2; no longer C45.2
- net VCC: now also U21.14 (VCC), U21.14 (VCC), U22.14 (VCC), U22.14 (VCC), C75.1
- net at C34.2, CN2.T: now also C33.2, R36.2
- net at C35.2, CN2.R: now also C32.2, R37.2
- now unconnected: U13.19 (NC), U13.22 (NC), U13.8 (NC), U13.9 (NC)
Other:
- note added: "ADDRESS SELECTOR"
- note added: "AUDIO OUTPUT"
- note added: "BUS BUFFERS"
- note added: "DSP"
- note added: "ISA BUS"
- note added: "POWER"
- note removed: "ANTIALIAS FILTER (OUTPUT)"
- note removed: "AUDIO POWER AMPLIFIER"
- note removed: "CURRENT TO VOLTAGE CONVERTER"
- note removed: "MUTE CIRCUIT"
- moved on the sheet: C1, C10, C11, C12, C13, C14, C15, C16, C17, C18, C19, C2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
